File: 02_vco_as3340/schematics/02_vco_as3340.kicad_pcb (KiCad board)
At the start: 2 copper layers, 75 x 100 mm, 89 parts, among them J1 Header 1, J10 SINE OUT, J2 Header 2, J3 SYNC IN, J4 FM IN, J5 PWM CV IN, J6 1V per O IN, J7 SQUARE OUT, J8 SAW OUT, J9 TRI OUT, Q1 BC547C, Q2 BC547C, U1 TL072, U2 AS3340, U3 TL074

Commit message: final tweaks
Connections:
- C12 pad 1: Net-(C12-Pad1) -> GND
- C13 pad 2: Net-(C12-Pad1) -> GND
- C18 pad 1: Net-(C18-Pad1) -> GND
- C19 pad 2: Net-(C18-Pad1) -> GND
Routing:
- net GND: track 378.6 -> 437.2 mm
- net Net-(C18-Pad1): track 24.5 -> 0.00 mm, vias 1 -> 0
- net Net-(C12-Pad1): track 14.3 -> 0.00 mm
