File: 02_vco_as3340/schematics/02_vco_as3340.kicad_sch (KiCad schematic)
At the start: 89 parts, among them J1 Header 1, J10 SINE OUT, J2 Header 2, J3 SYNC IN, J4 FM IN, J5 PWM CV IN, J6 1V per O IN, J7 SQUARE OUT, J8 SAW OUT, J9 TRI OUT, Q1 BC547C, Q2 BC547C, U1 TL072, U2 AS3340, U3 TL074

Commit message: 02 SMD!
Parts:
- removed C10, C11: 100nF, Capacitor_THT:C_Disc_D6.0mm_W2.5mm_P5.00mm, symbol Device:C_Small
- removed J1: Header 1, Connector_PinSocket_2.54mm:PinSocket_2x05_P2.54mm_Vertical, symbol Connector_Generic:Conn_02x05_Odd_Even
- removed J2: Header 2, Connector_PinSocket_2.54mm:PinSocket_2x04_P2.54mm_Vertical, symbol Connector_Generic:Conn_02x04_Odd_Even
- removed Q1, Q2: BC547C, Package_TO_SOT_THT:TO-92_Inline, symbol Transistor_BJT:2N3904
- added Q1, Q2: BC847, Package_TO_SOT_SMD:SOT-23, symbol Transistor_BJT:BC847
- added R49: 51k, cynthia:R SMD 0805, symbol Device:R_Small
- added R50: 1M, cynthia:R SMD 0805, symbol Device:R_Small
- added RV1: 250k, cynthia:potientiometer, symbol Device:R_Potentiometer_Small
- added RV2, RV3, RV4, RV5: 100k, cynthia:potientiometer, symbol Device:R_Potentiometer_Small
- added SW1: (no value), cynthia:switch_linear_1x4, symbol cynthia:switch_linear_1x4
- added SW2: SW_SPDT, cynthia:switch, symbol Switch:SW_SPDT
- added TP5, TP6, TP7, TP8: TestPoint, TestPoint:TestPoint_Pad_1.0x1.0mm, symbol Connector:TestPoint
- C1, C12, C13, C14, C17, C18, C19, C2, C3, C4, C5, C6, C9: footprint Capacitor_THT:C_Disc_D6.0mm_W2.5mm_P5.00mm -> cynthia:C SMD 0805
- C15, C16: footprint Capacitor_THT:C_Disc_D6.0mm_W2.5mm_P5.00mm -> Capacitor_THT:C_Disc_D10.5mm_W5.0mm_P10.00mm
- D1, D2: footprint Diode_THT:D_DO-35_SOD27_P7.62mm_Horizontal -> cynthia:C SMD 0805
- H1: footprint Connector_PinHeader_2.54mm:PinHeader_2x05_P2.54mm_Vertical -> cynthia:Eurorack Header
- J10, J7, J8, J9: footprint cynthia:6.35 mm jack socket mono in 3 pin socket tip pin west -> cynthia:3.5mm jack mono switched; symbol cynthia:6.35_mm_jack_socket_mono -> Connector_Audio:AudioJack2_SwitchT
- J3, J4, J5, J6: footprint cynthia:6.35 mm jack socket mono switched in 5 pin socket -> cynthia:3.5mm jack mono switched; symbol cynthia:6.35_mm_jack_socket_mono_switched -> Connector_Audio:AudioJack2_SwitchT
- R1, R10, R11, R12, R13, R14, R15, R16, R17, R18, R19, R2, R20, R21, R22, R23, R24, R25, R26, R27, R28, R29, R3, R30, R31, R32, R33, R34, R35, R36, R37, R39, R4, R40, R41, R42, R43, R44, R45, R46, R47, R48, R5, R6, R7, R8, R9: footprint Resistor_THT:R_Axial_DIN0207_L6.3mm_D2.5mm_P10.16mm_Horizontal -> cynthia:R SMD 0805
- R38: value 82k -> 100k; footprint Resistor_THT:R_Axial_DIN0207_L6.3mm_D2.5mm_P10.16mm_Horizontal -> cynthia:R SMD 0805
- TP1, TP2, TP3, TP4: footprint Potentiometer_THT:Potentiometer_Vishay_T73XW_Horizontal -> cynthia:trimmer
- U1: footprint Package_DIP:DIP-8_W7.62mm_Socket -> cynthia:SOIC-8_3.9x4.9mm_P1.27mm
- U2: footprint Package_DIP:DIP-16_W7.62mm_Socket -> cynthia:SOIC-16_3.9x9.9mm_P1.27mm
- U3: footprint Package_DIP:DIP-14_W7.62mm_Socket -> cynthia:SOIC-14_3.9x8.7mm_P1.27mm
Connections:
- net Mode LFO is gone; now on net GND: C15.1
- net Mode VCO is gone; now on net GND: C16.2
- net +12V: now also RV1.3, RV4.3, RV5.3
- net -12V: now also RV1.1, RV4.1, RV5.1
- net GND: now also R49.1, R50.1, RV2.1, RV3.1; no longer C15.2, C16.1
- net at R34.2, U2.10 (VTO): now also TP5.1
- net at R28.1, U2.4 (VP): now also R49.2, TP7.1
- net at R18.2, U1.7, U2.5 (VPWM): now also TP8.1
- net at R31.1, U2.8 (VSO): now also TP6.1
- net at C4.1, U2.9 (VSSI): now also R50.2
- net at R42.1: now also Q2.1 (B)
- net at R28.2, R38.1: now also U3.6 (-); no longer U3.2 (-)
- net at R38.2, R43.1: now also U3.7; no longer U3.1
- net at R39.2, R44.1: now also U3.1; no longer U3.7
- net at R26.2, R27.1: now also U3.5 (+); no longer U3.3 (+)
- net at R35.2, R37.2: now also Q2.2 (E)
- net at R41.2, R46.1, U3.12 (+): now also Q2.3 (C)
- net at R25.1, R35.1: now also Q1.2 (E)
- net at R23.1, TP4.1: now also Q1.1 (B)
- net at R24.2, R47.1, U3.13 (-): now also Q1.3 (C)
- net at R29.2, R30.1: now also U3.3 (+); no longer U3.5 (+)
- net at R31.2, R39.1: now also U3.2 (-); no longer U3.6 (-)
- net Coarse Tuning: no longer names the net of R4.1
- net Coarse Tuning: now also RV5.2
- net FM CV Hot: no longer names the net of J4.T
- net FM CV Hot: now also RV2.3
- net FM CV Levelled: no longer names the net of C5.2
- net FM CV Levelled: now also RV2.2
- net Fine Tuning: no longer names the net of R5.1
- net Fine Tuning: now also RV4.2
- net Hard Sync: no longer names the net of C2.2
- net Hard Sync: now also SW1.3
- net Hard Sync +: no longer names the net of C1.2
- net Hard Sync +: now also SW1.2
- net Hard Sync -: no longer names the net of C3.2
- net Hard Sync -: now also SW1.4
- net Mode COM: no longer names the net of U2.11 (CAP)
- net Mode COM: now also SW2.2 (B)
- net PWM CV Hot: no longer names the net of J5.T
- net PWM CV Hot: now also RV3.3
- net PWM CV Levelled: no longer names the net of R2.1
- net PWM CV Levelled: now also RV3.2
- net PWM Offset: no longer names the net of R1.1
- net PWM Offset: now also RV1.2
- net Soft Sync: no longer names the net of C4.2
- net Soft Sync: now also SW1.5
- net Sync COM: no longer names the net of J3.T
- net Sync COM: now also SW1.1
- new net: C15.2, SW2.1 (A)
- new net: C16.1, SW2.3 (C)
- no-connect marks 0 -> 4
Other:
- moved on the sheet: C17, C5, C6, R22, R3, R6, R8, R9
