File: 11_fm_drum/11_fm_drum.kicad_pcb (KiCad board)
At the start: 2 copper layers, 106 parts, among them J1 Conn_02x05_Odd_Even, J2 I/O, Q1 BC548, Q10 BC548, Q11 BC558, Q12 BC558, Q13 BC548, Q2 BC558, Q3 BC558, Q4 BC548, Q5 BC548, Q6 BC548, Q7 BC548, Q8 BC548, Q9 BC558, SW1 SW_SPDT, SW2 SW_SPDT, U1 TL074, U2 TL072

Commit message: split 11 into two boards
Parts:
- removed R17: 100k, Resistor_THT:R_Axial_DIN0207_L6.3mm_D2.5mm_P10.16mm_Horizontal
- removed R7: 1M, Resistor_THT:R_Axial_DIN0207_L6.3mm_D2.5mm_P10.16mm_Horizontal
- removed RV1, RV2, RV3: 100k, Potentiometer_THT:Potentiometer_Bourns_PTV09A-1_Single_Vertical
- removed RV4: 500k, Potentiometer_THT:Potentiometer_Bourns_PTV09A-1_Single_Vertical
- removed RV5: 1M, Potentiometer_THT:Potentiometer_Bourns_PTV09A-1_Single_Vertical
- removed RV7: 2M, Potentiometer_THT:Potentiometer_Bourns_3386W_Horizontal
- removed SW1, SW2: SW_SPDT, Connector_PinHeader_2.54mm:PinHeader_1x03_P2.54mm_Vertical
- added D15: 1N4148, Diode_THT:D_DO-35_SOD27_P7.62mm_Horizontal, F.Cu at (197.4, 123.9)
- added D16: 1N4148, Diode_THT:D_DO-35_SOD27_P7.62mm_Horizontal, F.Cu at (197.4, 127.5)
- added D17: 1N4148, Diode_THT:D_DO-35_SOD27_P7.62mm_Horizontal, F.Cu at (197.4, 131.0)
- added D18: 1N4148, Diode_THT:D_DO-35_SOD27_P7.62mm_Horizontal, F.Cu at (197.4, 134.6)
- added J3: Gate IN, cynthia:6.25mm Jack Stereo Switched, F.Cu at (125.5, 45.5)
- added J4: Acceent CV, cynthia:6.25mm Jack Stereo Switched, F.Cu at (125.5, 155.5)
- added J5: Tune CV, cynthia:6.25mm Jack Stereo Switched, F.Cu at (147.5, 45.5)
- added J6: Decay CV, cynthia:6.25mm Jack Stereo Switched, F.Cu at (170.5, 45.5)
- added J7: Out, cynthia:6.25mm Jack Stereo Switched, F.Cu at (171.5, 155.5)
- added R37: 2k, cynthia:R_Axial_DIN0207_L6.3mm_D2.5mm_P10.16mm_Horizontal, F.Cu at (81.9, 55.9)
- added R51: 470k, cynthia:R_Axial_DIN0207_L6.3mm_D2.5mm_P10.16mm_Horizontal, F.Cu at (95.2, 59.9)
- added R52: 1k, cynthia:R_Axial_DIN0207_L6.3mm_D2.5mm_P10.16mm_Horizontal, F.Cu at (95.2, 64.0)
- C1: value 2.2nF -> 10nF; footprint Capacitor_THT:C_Rect_L7.2mm_W5.5mm_P5.00mm_FKS2_FKP2_MKS2_MKP2 -> Capacitor_THT:C_Rect_L7.2mm_W3.5mm_P5.00mm_FKS2_FKP2_MKS2_MKP2
- C10: value 47nF -> 100nF; footprint Capacitor_THT:CP_Radial_D7.5mm_P2.50mm -> Capacitor_THT:C_Disc_D7.5mm_W2.5mm_P5.00mm
- C11: value 47nF -> 5.6nF; footprint Capacitor_THT:CP_Radial_D7.5mm_P2.50mm -> Capacitor_THT:C_Rect_L7.2mm_W3.5mm_P5.00mm_FKS2_FKP2_MKS2_MKP2
- C12, C14: value 100nF -> 470pF; footprint Capacitor_THT:C_Disc_D7.5mm_W2.5mm_P5.00mm -> Capacitor_THT:C_Rect_L7.2mm_W3.5mm_P5.00mm_FKS2_FKP2_MKS2_MKP2
- C13: value 100nF -> 2.2nF; footprint Capacitor_THT:C_Disc_D7.5mm_W2.5mm_P5.00mm -> Capacitor_THT:C_Rect_L7.2mm_W3.5mm_P5.00mm_FKS2_FKP2_MKS2_MKP2
- C15: value 100nF -> 15nF; footprint Capacitor_THT:C_Disc_D7.5mm_W2.5mm_P5.00mm -> Capacitor_THT:C_Rect_L7.2mm_W3.5mm_P5.00mm_FKS2_FKP2_MKS2_MKP2
- C16: value 100nF -> 1uF; footprint Capacitor_THT:C_Disc_D7.5mm_W2.5mm_P5.00mm -> Capacitor_THT:C_Rect_L7.2mm_W5.5mm_P5.00mm_FKS2_FKP2_MKS2_MKP2
- C17: value 100nF -> 330pF; footprint Capacitor_THT:C_Disc_D7.5mm_W2.5mm_P5.00mm -> Capacitor_THT:C_Rect_L7.2mm_W3.5mm_P5.00mm_FKS2_FKP2_MKS2_MKP2
- C2: value 330pF -> 47uF; footprint Capacitor_THT:C_Rect_L7.2mm_W5.5mm_P5.00mm_FKS2_FKP2_MKS2_MKP2 -> Capacitor_THT:CP_Radial_D7.5mm_P2.50mm
- C3: value 5.6nF -> 47uF; footprint Capacitor_THT:C_Rect_L7.2mm_W5.5mm_P5.00mm_FKS2_FKP2_MKS2_MKP2 -> Capacitor_THT:CP_Radial_D7.5mm_P2.50mm
- C4: value 470pF -> 470nF
- C5: value 470pF -> 100nF; footprint Capacitor_THT:C_Rect_L7.2mm_W5.5mm_P5.00mm_FKS2_FKP2_MKS2_MKP2 -> Capacitor_THT:C_Disc_D7.5mm_W2.5mm_P5.00mm
- C6: value 15nF -> 100nF; footprint Capacitor_THT:C_Rect_L7.2mm_W5.5mm_P5.00mm_FKS2_FKP2_MKS2_MKP2 -> Capacitor_THT:C_Disc_D7.5mm_W2.5mm_P5.00mm
- C7: value 1uF -> 100nF; footprint Capacitor_THT:C_Rect_L7.2mm_W5.5mm_P5.00mm_FKS2_FKP2_MKS2_MKP2 -> Capacitor_THT:C_Disc_D7.5mm_W2.5mm_P5.00mm
- C8: value 10nF -> 100nF; footprint Capacitor_THT:C_Rect_L7.2mm_W5.5mm_P5.00mm_FKS2_FKP2_MKS2_MKP2 -> Capacitor_THT:C_Disc_D7.5mm_W2.5mm_P5.00mm
- C9: value 470nF -> 100nF; footprint Capacitor_THT:C_Rect_L7.2mm_W5.5mm_P5.00mm_FKS2_FKP2_MKS2_MKP2 -> Capacitor_THT:C_Disc_D7.5mm_W2.5mm_P5.00mm
- J1: moved to B.Cu
- J2: value I/O -> Conn_02x10_Counter_Clockwise; footprint Connector_PinHeader_2.54mm:PinHeader_1x05_P2.54mm_Vertical -> Connector_PinSocket_2.54mm:PinSocket_2x10_P2.54mm_Vertical
- Q1, Q13, Q5, Q7: value BC548 -> BC558
- Q11, Q12, Q2, Q9: value BC558 -> BC548
- R1, R11, R15, R20, R28, R31, R44, R5: footprint Resistor_THT:R_Axial_DIN0207_L6.3mm_D2.5mm_P10.16mm_Horizontal -> cynthia:R_Axial_DIN0207_L6.3mm_D2.5mm_P10.16mm_Horizontal
- R10: value 51k -> 3.3; footprint Resistor_THT:R_Axial_DIN0207_L6.3mm_D2.5mm_P10.16mm_Horizontal -> cynthia:R_Axial_DIN0207_L6.3mm_D2.5mm_P10.16mm_Horizontal
- R12, R27, R46: value 100k -> 10k; footprint Resistor_THT:R_Axial_DIN0207_L6.3mm_D2.5mm_P10.16mm_Horizontal -> cynthia:R_Axial_DIN0207_L6.3mm_D2.5mm_P10.16mm_Horizontal
- R13: value 100k -> 2k; footprint Resistor_THT:R_Axial_DIN0207_L6.3mm_D2.5mm_P10.16mm_Horizontal -> cynthia:R_Axial_DIN0207_L6.3mm_D2.5mm_P10.16mm_Horizontal
- R14: value 51k -> 470k; footprint Resistor_THT:R_Axial_DIN0207_L6.3mm_D2.5mm_P10.16mm_Horizontal -> cynthia:R_Axial_DIN0207_L6.3mm_D2.5mm_P10.16mm_Horizontal
- R16, R4: value 100k -> 39k; footprint Resistor_THT:R_Axial_DIN0207_L6.3mm_D2.5mm_P10.16mm_Horizontal -> cynthia:R_Axial_DIN0207_L6.3mm_D2.5mm_P10.16mm_Horizontal
- R18: value 10k -> 33k; footprint Resistor_THT:R_Axial_DIN0207_L6.3mm_D2.5mm_P10.16mm_Horizontal -> cynthia:R_Axial_DIN0207_L6.3mm_D2.5mm_P10.16mm_Horizontal
- R19: value 68k -> 100k; footprint Resistor_THT:R_Axial_DIN0207_L6.3mm_D2.5mm_P10.16mm_Horizontal -> cynthia:R_Axial_DIN0207_L6.3mm_D2.5mm_P10.16mm_Horizontal
- R2: value 100k -> 33k; footprint Resistor_THT:R_Axial_DIN0207_L6.3mm_D2.5mm_P10.16mm_Horizontal -> cynthia:R_Axial_DIN0207_L6.3mm_D2.5mm_P10.16mm_Horizontal
- R21: value 33k -> 100k; footprint Resistor_THT:R_Axial_DIN0207_L6.3mm_D2.5mm_P10.16mm_Horizontal -> cynthia:R_Axial_DIN0207_L6.3mm_D2.5mm_P10.16mm_Horizontal
- R22: value 100k -> 51k; footprint Resistor_THT:R_Axial_DIN0207_L6.3mm_D2.5mm_P10.16mm_Horizontal -> cynthia:R_Axial_DIN0207_L6.3mm_D2.5mm_P10.16mm_Horizontal
- R23, R45: value 10k -> 1M; footprint Resistor_THT:R_Axial_DIN0207_L6.3mm_D2.5mm_P10.16mm_Horizontal -> cynthia:R_Axial_DIN0207_L6.3mm_D2.5mm_P10.16mm_Horizontal
- R24, R33: value 2k -> 100k; footprint Resistor_THT:R_Axial_DIN0207_L6.3mm_D2.5mm_P10.16mm_Horizontal -> cynthia:R_Axial_DIN0207_L6.3mm_D2.5mm_P10.16mm_Horizontal
- R25: value 470k -> 10k; footprint Resistor_THT:R_Axial_DIN0207_L6.3mm_D2.5mm_P10.16mm_Horizontal -> cynthia:R_Axial_DIN0207_L6.3mm_D2.5mm_P10.16mm_Horizontal
- R26: value 39k -> 100k; footprint Resistor_THT:R_Axial_DIN0207_L6.3mm_D2.5mm_P10.16mm_Horizontal -> cynthia:R_Axial_DIN0207_L6.3mm_D2.5mm_P10.16mm_Horizontal
- R29: value 200k -> 100k; footprint Resistor_THT:R_Axial_DIN0207_L6.3mm_D2.5mm_P10.16mm_Horizontal -> cynthia:R_Axial_DIN0207_L6.3mm_D2.5mm_P10.16mm_Horizontal
- R3: value 100k -> 470; footprint Resistor_THT:R_Axial_DIN0207_L6.3mm_D2.5mm_P10.16mm_Horizontal -> cynthia:R_Axial_DIN0207_L6.3mm_D2.5mm_P10.16mm_Horizontal
- R30: value 10k -> 200k; footprint Resistor_THT:R_Axial_DIN0207_L6.3mm_D2.5mm_P10.16mm_Horizontal -> cynthia:R_Axial_DIN0207_L6.3mm_D2.5mm_P10.16mm_Horizontal
- R32: value 18k -> 100k; footprint Resistor_THT:R_Axial_DIN0207_L6.3mm_D2.5mm_P10.16mm_Horizontal -> cynthia:R_Axial_DIN0207_L6.3mm_D2.5mm_P10.16mm_Horizontal
- R34: value 47 -> 18k; footprint Resistor_THT:R_Axial_DIN0207_L6.3mm_D2.5mm_P10.16mm_Horizontal -> cynthia:R_Axial_DIN0207_L6.3mm_D2.5mm_P10.16mm_Horizontal
- R35, R41: value 470k -> 100k; footprint Resistor_THT:R_Axial_DIN0207_L6.3mm_D2.5mm_P10.16mm_Horizontal -> cynthia:R_Axial_DIN0207_L6.3mm_D2.5mm_P10.16mm_Horizontal
- R36: value 1M -> 100k; footprint Resistor_THT:R_Axial_DIN0207_L6.3mm_D2.5mm_P10.16mm_Horizontal -> cynthia:R_Axial_DIN0207_L6.3mm_D2.5mm_P10.16mm_Horizontal
- R38: value 200k -> 51k; footprint Resistor_THT:R_Axial_DIN0207_L6.3mm_D2.5mm_P10.16mm_Horizontal -> cynthia:R_Axial_DIN0207_L6.3mm_D2.5mm_P10.16mm_Horizontal
- R39: value 1k -> 1M; footprint Resistor_THT:R_Axial_DIN0207_L6.3mm_D2.5mm_P10.16mm_Horizontal -> cynthia:R_Axial_DIN0207_L6.3mm_D2.5mm_P10.16mm_Horizontal
- R40: value 4.7k -> 47; footprint Resistor_THT:R_Axial_DIN0207_L6.3mm_D2.5mm_P10.16mm_Horizontal -> cynthia:R_Axial_DIN0207_L6.3mm_D2.5mm_P10.16mm_Horizontal
- R42: value 33k -> 470k; footprint Resistor_THT:R_Axial_DIN0207_L6.3mm_D2.5mm_P10.16mm_Horizontal -> cynthia:R_Axial_DIN0207_L6.3mm_D2.5mm_P10.16mm_Horizontal
- R43: value 39k -> 1k; footprint Resistor_THT:R_Axial_DIN0207_L6.3mm_D2.5mm_P10.16mm_Horizontal -> cynthia:R_Axial_DIN0207_L6.3mm_D2.5mm_P10.16mm_Horizontal
- R47: value 5.6k -> 68k; footprint Resistor_THT:R_Axial_DIN0207_L6.3mm_D2.5mm_P10.16mm_Horizontal -> cynthia:R_Axial_DIN0207_L6.3mm_D2.5mm_P10.16mm_Horizontal
- R48: value 470 -> 200k; footprint Resistor_THT:R_Axial_DIN0207_L6.3mm_D2.5mm_P10.16mm_Horizontal -> cynthia:R_Axial_DIN0207_L6.3mm_D2.5mm_P10.16mm_Horizontal
- R49: value 47k -> 4.7k; footprint Resistor_THT:R_Axial_DIN0207_L6.3mm_D2.5mm_P10.16mm_Horizontal -> cynthia:R_Axial_DIN0207_L6.3mm_D2.5mm_P10.16mm_Horizontal
- R50: value 1k -> 100k; footprint Resistor_THT:R_Axial_DIN0207_L6.3mm_D2.5mm_P10.16mm_Horizontal -> cynthia:R_Axial_DIN0207_L6.3mm_D2.5mm_P10.16mm_Horizontal
- R6: value 10k -> 1k; footprint Resistor_THT:R_Axial_DIN0207_L6.3mm_D2.5mm_P10.16mm_Horizontal -> cynthia:R_Axial_DIN0207_L6.3mm_D2.5mm_P10.16mm_Horizontal
- R8: value 1M -> 10k; footprint Resistor_THT:R_Axial_DIN0207_L6.3mm_D2.5mm_P10.16mm_Horizontal -> cynthia:R_Axial_DIN0207_L6.3mm_D2.5mm_P10.16mm_Horizontal
- R9: value 33k -> 47k; footprint Resistor_THT:R_Axial_DIN0207_L6.3mm_D2.5mm_P10.16mm_Horizontal -> cynthia:R_Axial_DIN0207_L6.3mm_D2.5mm_P10.16mm_Horizontal
- RV6: value 1M -> 2M; footprint Potentiometer_THT:Potentiometer_Bourns_PTV09A-1_Single_Vertical -> cynthia:trimmer; moved to B.Cu
- U1: value TL074 -> TL072; footprint Package_DIP:DIP-14_W7.62mm_Socket -> Package_DIP:DIP-8_W7.62mm_Socket
- U2: value TL072 -> TL074; footprint Package_DIP:DIP-8_W7.62mm_Socket -> Package_DIP:DIP-14_W7.62mm_Socket
- moved RV6 269.1 mm to (180.0, 95.0), turned to 180 degrees
- moved D1 209.2 mm to (197.4, 74.2)
- moved D10 209.2 mm to (197.4, 106.2)
- moved D5 209.2 mm to (197.4, 88.4)
- moved D11 209.2 mm to (197.4, 109.7)
- moved D13 209.2 mm to (197.4, 116.8)
- moved D14 209.2 mm to (197.4, 120.3)
- moved D2 209.2 mm to (197.4, 77.8)
- moved D3 209.2 mm to (197.4, 81.3)
- moved D4 209.2 mm to (197.4, 84.8)
- moved D6 209.2 mm to (197.4, 92.0)
- moved D7 209.2 mm to (197.4, 95.5)
- moved D8 209.2 mm to (197.4, 99.0)
- moved D9 209.2 mm to (197.4, 102.6)
- moved C3 202.2 mm to (164.5, 25.0)
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Connections:
- C1 pad 1: Net-(SW1-A) -> gate in
- C1 pad 2: Net-(Q1-E) -> Net-(D2-K)
- C10 pad 1: +12V -> GND
- C10 pad 2: GND -> -12V
- C11 pad 1: GND -> Net-(D6-K)
- C11 pad 2: -12V -> GND
- C12 pad 1: +12V -> Net-(C12-Pad1)
- C12 pad 2: GND -> Net-(Q7-C)
- C13 pad 1: GND -> io fm on/off pin 1
- C13 pad 2: -12V -> Net-(Q8-E)
- C14 pad 1: +12V -> Net-(Q9-B)
- C14 pad 2: GND -> Net-(C12-Pad1)
- C15 pad 1: GND -> Net-(C15-Pad1)
- C15 pad 2: -12V -> Net-(Q9-E)
- C16 pad 1: +12V -> io decay pin 1
- C17 pad 1: GND -> triangle 2
- C17 pad 2: -12V -> Net-(Q11-E)
- C2 pad 1: triangle 2 -> +12V
- C2 pad 2: Net-(Q6-E) -> GND
- C3 pad 1: Net-(D5-K) -> GND
- C3 pad 2: GND -> -12V
- C4 pad 1: Net-(C4-Pad1) -> io tune decay 1
- C4 pad 2: Net-(Q9-C) -> GND
- C5 pad 1: Net-(Q8-B) -> +12V
- C5 pad 2: Net-(C4-Pad1) -> GND
- C6 pad 1: Net-(C6-Pad1) -> GND
- C6 pad 2: Net-(Q8-E) -> -12V
- C7 pad 1: Net-(D11-K) -> +12V
- C8 pad 1: gate in -> GND
- C8 pad 2: Net-(D12-K) -> -12V
- C9 pad 1: Net-(D13-K) -> +12V
- D1 pad 1: Net-(D1-K) -> io tune decay 1
- D10 pad 1: square 1 -> sine
- D10 pad 2: Net-(D10-A) -> GND
- D11 pad 2: accented trigger -> square 1
- D12 pad 1: Net-(D12-K) -> Net-(D11-K)
- D12 pad 2: GND -> square 2
- D13 pad 1: Net-(D13-K) -> square 1
- D14 pad 1: Net-(D14-K) -> square 2
- D14 pad 2: Net-(D13-K) -> Net-(D13-A)
- D2 pad 2: tune 2 -> GND
- D3 pad 1: sine -> +12V
- D3 pad 2: GND -> Net-(D3-A)
- D4 pad 1: GND -> Net-(D3-A)
- D4 pad 2: sine -> GND
- D5 pad 2: accented trigger -> io tune decay 1
- D6 pad 2: trigger -> accented trigger
- D7 pad 2: square 1 -> io tune lvl pin 2
- D8 pad 1: square 2 -> Net-(D8-K)
- D8 pad 2: Net-(D10-A) -> trigger
- D9 pad 1: Net-(D7-K) -> GND
- D9 pad 2: square 2 -> sine
- J2 pad 1: gate in -> tune cv
- J2 pad 2: accent cv -> io tune lvl pin 2
- J2 pad 3: tune cv -> io tune decay 1
- J2 pad 4: decay cv -> io tune depth 1
- J2 pad 5: out -> tune 2
- Q1 pad 1: Net-(Q1-C) -> GND
- Q1 pad 2: Net-(Q1-B) -> Net-(D3-A)
- Q10 pad 3: Net-(Q10-E) -> GND
- Q11 pad 1: GND -> Net-(Q11-C)
- Q11 pad 2: decay cv -> Net-(Q11-B)
- Q12 pad 1: GND -> Net-(Q12-C)
- Q12 pad 2: accent cv -> Net-(Q12-B)
- Q13 pad 1: +12V -> GND
- Q13 pad 2: Net-(Q13-B) -> Net-(D17-A)
- Q13 pad 3: accented trigger -> Net-(Q13-E)
- Q2 pad 1: GND -> +12V
- Q2 pad 2: Net-(D1-K) -> Net-(Q2-B)
- Q2 pad 3: Net-(Q2-E) -> accented trigger
- Q3 pad 2: Net-(D1-K) -> Net-(D7-K)
- Q3 pad 3: Net-(Q3-E) -> io tune 1 pin 3
- Q4 pad 3: GND -> sine
- Q5 pad 1: Net-(Q5-C) -> GND
- Q5 pad 2: Net-(Q5-B) -> Net-(D7-K)
- Q5 pad 3: GND -> io tune 2 pin 3
- Q6 pad 3: Net-(Q6-E) -> GND
- Q7 pad 3: sine -> Net-(D11-K)
- Q8 pad 1: +12V -> Net-(Q8-C)
- Q9 pad 1: Net-(Q9-C) -> +12V
- Q9 pad 3: Net-(D7-K) -> Net-(Q9-E)
- R1 pad 1: tune 1 -> GND
- R1 pad 2: Net-(Q1-E) -> gate in
- R10 pad 1: Net-(Q4-C) -> Net-(Q1-E)
- R10 pad 2: Net-(Q1-E) -> Net-(Q2-B)
- R11 pad 1: Net-(Q4-B) -> GND
- R11 pad 2: square 1 -> accented trigger
- R12 pad 1: Net-(D2-K) -> triangle 2
- R12 pad 2: Net-(Q6-E) -> sine
- R13 pad 1: Net-(D2-K) -> triangle 2
- R13 pad 2: Net-(U1C-+) -> Net-(Q4-C)
- R14 pad 1: Net-(Q5-C) -> Net-(D6-K)
- R14 pad 2: Net-(Q6-E) -> Net-(Q4-B)
- R15 pad 1: trigger -> -12V
- R15 pad 2: Net-(Q6-B) -> Net-(D7-K)
- R16 pad 1: GND -> Net-(D8-K)
- R16 pad 2: Net-(U1C-+) -> sine
- R18 pad 1: Net-(Q6-C) -> io tune 2 pin 2
- R18 pad 2: triangle 2 -> tune 2
- R19 pad 1: GND -> tune 1
- R19 pad 2: Net-(U1D-+) -> Net-(Q8-E)
- R2 pad 1: tune 1 -> GND
- R2 pad 2: Net-(U1A-+) -> Net-(U1A--)
- R20 pad 1: Net-(U1D-+) -> tune 1
- R20 pad 2: square 2 -> Net-(U2A-+)
- R21 pad 1: Net-(R21-Pad1) -> Net-(D13-A)
- R21 pad 2: tune 2 -> Net-(Q7-B)
- R22 pad 1: Net-(SW1-B) -> Net-(Q6-C)
- R22 pad 2: tune 2 -> Net-(Q8-E)
- R23 pad 1: triangle 2 -> trigger
- R23 pad 2: sine -> Net-(Q8-B)
- R24 pad 1: triangle 2 -> GND
- R24 pad 2: Net-(Q7-C) -> Net-(U2A-+)
- R25 pad 1: Net-(D5-K) -> -12V
- R25 pad 2: Net-(Q7-B) -> Net-(Q7-C)
- R26 pad 1: Net-(D6-K) -> Net-(Q6-B)
- R26 pad 2: sine -> square 1
- R27 pad 1: Net-(D10-A) -> Net-(Q8-C)
- R27 pad 2: Net-(Q9-B) -> io fm on/off pin 1
- R28 pad 1: -12V -> Net-(Q9-E)
- R28 pad 2: Net-(Q9-C) -> Net-(C12-Pad1)
- R29 pad 2: Net-(Q8-B) -> Net-(U2B-+)
- R3 pad 1: GND -> trigger
- R3 pad 2: Net-(U1A-+) -> Net-(D1-A)
- R30 pad 1: -12V -> GND
- R30 pad 2: Net-(Q8-E) -> Net-(Q9-B)
- R31 pad 1: Net-(Q8-E) -> -12V
- R31 pad 2: Net-(C4-Pad1) -> Net-(Q9-E)
- R32 pad 1: Net-(C6-Pad1) -> Net-(U2B-+)
- R32 pad 2: pulse -> square 1
- R33 pad 1: Net-(SW2-B) -> io fm on/off pin 2
- R33 pad 2: Net-(Q10-C) -> tune 2
- R34 pad 1: GND -> Net-(C15-Pad1)
- R34 pad 2: Net-(Q10-C) -> pulse
- R35 pad 1: Net-(D11-K) -> Net-(D15-K)
- R35 pad 2: Net-(Q10-B) -> Net-(Q11-E)
- R36 pad 1: Net-(D11-K) -> Net-(D15-K)
- R36 pad 2: Net-(R36-Pad2) -> Net-(U2C-+)
- R38 pad 1: Net-(Q10-E) -> Net-(Q10-C)
- R38 pad 2: Net-(R38-Pad2) -> Net-(Q11-E)
- R39 pad 1: Net-(R38-Pad2) -> trigger
- R39 pad 2: out -> Net-(Q11-B)
- R4 pad 2: Net-(U1B-+) -> Net-(D2-K)
- R40 pad 1: Net-(R40-Pad1) -> GND
- R40 pad 2: Net-(Q11-E) -> Net-(Q12-C)
- R41 pad 2: Net-(Q11-E) -> Net-(U2C-+)
- R42 pad 1: GND -> io decay pin 1
- R42 pad 2: Net-(U2A--) -> Net-(Q12-B)
- R43 pad 1: GND -> decay cv
- R43 pad 2: Net-(D12-K) -> Net-(D17-A)
- R44 pad 1: Net-(U2A--) -> Net-(Q10-B)
- R44 pad 2: +12V -> square 2
- R45 pad 1: trigger -> io decay pin 1
- R45 pad 2: Net-(Q13-B) -> Net-(R45-Pad2)
- R46 pad 1: GND -> Net-(Q11-C)
- R46 pad 2: accented trigger -> triangle 2
- R47 pad 1: Net-(Q12-E) -> GND
- R47 pad 2: Net-(Q13-B) -> Net-(U2D-+)
- R48 pad 1: trigger -> Net-(Q12-E)
- R48 pad 2: Net-(D13-A) -> Net-(R48-Pad2)
- R49 pad 1: Net-(D14-K) -> Net-(Q13-E)
- R49 pad 2: Net-(R49-Pad2) -> io decay pin 2
- R5 pad 1: Net-(U1B-+) -> Net-(U1A--)
- R5 pad 2: square 1 -> +12V
- R50 pad 1: GND -> Net-(U2D-+)
- R50 pad 2: Net-(R50-Pad2) -> square 2
- R6 pad 1: Net-(Q1-C) -> accent cv
- R6 pad 2: Net-(SW1-A) -> Net-(D3-A)
- R8 pad 1: GND -> trigger
- R8 pad 2: Net-(D1-K) -> Net-(Q2-B)
- R9 pad 1: Net-(R9-Pad1) -> Net-(D5-K)
- R9 pad 2: +12V -> io tune depth 1
- RV6 pad 1: Net-(D13-K) -> Net-(Q12-E)
- RV6 pad 2: Net-(R50-Pad2) -> Net-(R45-Pad2)
- RV6 pad 3: Net-(R50-Pad2) -> Net-(R45-Pad2)
- U1 pad 1: Net-(SW1-A) -> trigger
- U1 pad 2: Net-(Q1-E) -> Net-(U1A--)
- U1 pad 3: Net-(U1A-+) -> Net-(D2-K)
- U1 pad 4: +12V -> -12V
- U1 pad 5: Net-(U1B-+) -> GND
- U1 pad 6: Net-(SW1-A) -> Net-(Q12-E)
- U1 pad 7: square 1 -> Net-(R48-Pad2)
- U1 pad 8: triangle 2 -> +12V
- U2 pad 1: trigger -> io fm on/off pin 1
- U2 pad 2: Net-(U2A--) -> Net-(Q8-E)
- U2 pad 3: Net-(D12-K) -> Net-(U2A-+)
- U2 pad 4: -12V -> +12V
- U2 pad 5: GND -> Net-(U2B-+)
- U2 pad 6: Net-(Q10-E) -> io fm on/off pin 1
- U2 pad 7: Net-(R38-Pad2) -> square 1
- U2 pad 8: +12V -> triangle 2
