File: 11_fm_drum/11_fm_drum.kicad_sch (KiCad schematic)
At the start: 106 parts, among them J1 Conn_02x05_Odd_Even, J2 I/O, Q1 BC548, Q10 BC548, Q11 BC558, Q12 BC558, Q13 BC548, Q2 BC558, Q3 BC558, Q4 BC548, Q5 BC548, Q6 BC548, Q7 BC548, Q8 BC548, Q9 BC558, SW1 SW_SPDT, SW2 SW_SPDT, U1 TL074, U2 TL072

Commit message: split 11 into two boards
Parts:
- removed J2: I/O, Connector_PinHeader_2.54mm:PinHeader_1x05_P2.54mm_Vertical, symbol Connector:Conn_01x05_Pin
- removed R50: 1k, Resistor_THT:R_Axial_DIN0207_L6.3mm_D2.5mm_P10.16mm_Horizontal, symbol Device:R
- removed R9: 33k, Resistor_THT:R_Axial_DIN0207_L6.3mm_D2.5mm_P10.16mm_Horizontal, symbol Device:R
- removed RV1, RV2, RV3: 100k, Potentiometer_THT:Potentiometer_Bourns_PTV09A-1_Single_Vertical, symbol Device:R_Potentiometer
- removed RV4: 500k, Potentiometer_THT:Potentiometer_Bourns_PTV09A-1_Single_Vertical, symbol Device:R_Potentiometer
- removed RV5, RV6: 1M, Potentiometer_THT:Potentiometer_Bourns_PTV09A-1_Single_Vertical, symbol Device:R_Potentiometer
- removed SW1, SW2: SW_SPDT, Connector_PinHeader_2.54mm:PinHeader_1x03_P2.54mm_Vertical, symbol Switch:SW_SPDT
- added D17, D18, D3, D4: 1N4148, Diode_THT:D_DO-35_SOD27_P7.62mm_Horizontal, symbol Diode:1N4148
- added J2: Conn_02x10_Counter_Clockwise, Connector_PinSocket_2.54mm:PinSocket_2x10_P2.54mm_Vertical, symbol Connector_Generic:Conn_02x10_Counter_Clockwise
- added J3: Gate IN, cynthia:6.25mm Jack Stereo Switched, symbol cynthia:6.35_mm_jack_socket_stereo_switched
- added J4: Acceent CV, cynthia:6.25mm Jack Stereo Switched, symbol cynthia:6.35_mm_jack_socket_stereo_switched
- added J5: Tune CV, cynthia:6.25mm Jack Stereo Switched, symbol cynthia:6.35_mm_jack_socket_stereo_switched
- added J6: Decay CV, cynthia:6.25mm Jack Stereo Switched, symbol cynthia:6.35_mm_jack_socket_stereo_switched
- added J7: Out, cynthia:6.25mm Jack Stereo Switched, symbol cynthia:6.35_mm_jack_socket_stereo_switched
- added R1: 100k, cynthia:R_Axial_DIN0207_L6.3mm_D2.5mm_P10.16mm_Horizontal, symbol Device:R
- added R43, R6: 1k, cynthia:R_Axial_DIN0207_L6.3mm_D2.5mm_P10.16mm_Horizontal, symbol Device:R
- C1: renamed from C8; footprint Capacitor_THT:C_Rect_L7.2mm_W5.5mm_P5.00mm_FKS2_FKP2_MKS2_MKP2 -> Capacitor_THT:C_Rect_L7.2mm_W3.5mm_P5.00mm_FKS2_FKP2_MKS2_MKP2
- C11: renamed from C3; footprint Capacitor_THT:C_Rect_L7.2mm_W5.5mm_P5.00mm_FKS2_FKP2_MKS2_MKP2 -> Capacitor_THT:C_Rect_L7.2mm_W3.5mm_P5.00mm_FKS2_FKP2_MKS2_MKP2
- C12: renamed from C4; footprint Capacitor_THT:C_Rect_L7.2mm_W5.5mm_P5.00mm_FKS2_FKP2_MKS2_MKP2 -> Capacitor_THT:C_Rect_L7.2mm_W3.5mm_P5.00mm_FKS2_FKP2_MKS2_MKP2
- C13: renamed from C1; footprint Capacitor_THT:C_Rect_L7.2mm_W5.5mm_P5.00mm_FKS2_FKP2_MKS2_MKP2 -> Capacitor_THT:C_Rect_L7.2mm_W3.5mm_P5.00mm_FKS2_FKP2_MKS2_MKP2
- C14: renamed from C5; footprint Capacitor_THT:C_Rect_L7.2mm_W5.5mm_P5.00mm_FKS2_FKP2_MKS2_MKP2 -> Capacitor_THT:C_Rect_L7.2mm_W3.5mm_P5.00mm_FKS2_FKP2_MKS2_MKP2
- C15: renamed from C6; footprint Capacitor_THT:C_Rect_L7.2mm_W5.5mm_P5.00mm_FKS2_FKP2_MKS2_MKP2 -> Capacitor_THT:C_Rect_L7.2mm_W3.5mm_P5.00mm_FKS2_FKP2_MKS2_MKP2
- C17: renamed from C2; footprint Capacitor_THT:C_Rect_L7.2mm_W5.5mm_P5.00mm_FKS2_FKP2_MKS2_MKP2 -> Capacitor_THT:C_Rect_L7.2mm_W3.5mm_P5.00mm_FKS2_FKP2_MKS2_MKP2
- C2: renamed from C10; value 47nF -> 47uF
- C3: renamed from C11; value 47nF -> 47uF
- R10: renamed from R47; value 5.6k -> 3.3; footprint Resistor_THT:R_Axial_DIN0207_L6.3mm_D2.5mm_P10.16mm_Horizontal -> cynthia:R_Axial_DIN0207_L6.3mm_D2.5mm_P10.16mm_Horizontal
- R11: renamed from R46; footprint Resistor_THT:R_Axial_DIN0207_L6.3mm_D2.5mm_P10.16mm_Horizontal -> cynthia:R_Axial_DIN0207_L6.3mm_D2.5mm_P10.16mm_Horizontal
- R12: renamed from R23; footprint Resistor_THT:R_Axial_DIN0207_L6.3mm_D2.5mm_P10.16mm_Horizontal -> cynthia:R_Axial_DIN0207_L6.3mm_D2.5mm_P10.16mm_Horizontal
- R13: renamed from R24; footprint Resistor_THT:R_Axial_DIN0207_L6.3mm_D2.5mm_P10.16mm_Horizontal -> cynthia:R_Axial_DIN0207_L6.3mm_D2.5mm_P10.16mm_Horizontal
- R14: renamed from R25; footprint Resistor_THT:R_Axial_DIN0207_L6.3mm_D2.5mm_P10.16mm_Horizontal -> cynthia:R_Axial_DIN0207_L6.3mm_D2.5mm_P10.16mm_Horizontal
- R15: renamed from R8; footprint Resistor_THT:R_Axial_DIN0207_L6.3mm_D2.5mm_P10.16mm_Horizontal -> cynthia:R_Axial_DIN0207_L6.3mm_D2.5mm_P10.16mm_Horizontal
- R16: renamed from R26; footprint Resistor_THT:R_Axial_DIN0207_L6.3mm_D2.5mm_P10.16mm_Horizontal -> cynthia:R_Axial_DIN0207_L6.3mm_D2.5mm_P10.16mm_Horizontal
- R18: renamed from R21; footprint Resistor_THT:R_Axial_DIN0207_L6.3mm_D2.5mm_P10.16mm_Horizontal -> cynthia:R_Axial_DIN0207_L6.3mm_D2.5mm_P10.16mm_Horizontal
- R19: renamed from R1; footprint Resistor_THT:R_Axial_DIN0207_L6.3mm_D2.5mm_P10.16mm_Horizontal -> cynthia:R_Axial_DIN0207_L6.3mm_D2.5mm_P10.16mm_Horizontal
- R2: renamed from R42; footprint Resistor_THT:R_Axial_DIN0207_L6.3mm_D2.5mm_P10.16mm_Horizontal -> cynthia:R_Axial_DIN0207_L6.3mm_D2.5mm_P10.16mm_Horizontal
- R20: renamed from R2; footprint Resistor_THT:R_Axial_DIN0207_L6.3mm_D2.5mm_P10.16mm_Horizontal -> cynthia:R_Axial_DIN0207_L6.3mm_D2.5mm_P10.16mm_Horizontal
- R21: renamed from R27; footprint Resistor_THT:R_Axial_DIN0207_L6.3mm_D2.5mm_P10.16mm_Horizontal -> cynthia:R_Axial_DIN0207_L6.3mm_D2.5mm_P10.16mm_Horizontal
- R22: renamed from R10; footprint Resistor_THT:R_Axial_DIN0207_L6.3mm_D2.5mm_P10.16mm_Horizontal -> cynthia:R_Axial_DIN0207_L6.3mm_D2.5mm_P10.16mm_Horizontal
- R23: renamed from R7; footprint Resistor_THT:R_Axial_DIN0207_L6.3mm_D2.5mm_P10.16mm_Horizontal -> cynthia:R_Axial_DIN0207_L6.3mm_D2.5mm_P10.16mm_Horizontal
- R24: renamed from R3; footprint Resistor_THT:R_Axial_DIN0207_L6.3mm_D2.5mm_P10.16mm_Horizontal -> cynthia:R_Axial_DIN0207_L6.3mm_D2.5mm_P10.16mm_Horizontal
- R25: renamed from R28; footprint Resistor_THT:R_Axial_DIN0207_L6.3mm_D2.5mm_P10.16mm_Horizontal -> cynthia:R_Axial_DIN0207_L6.3mm_D2.5mm_P10.16mm_Horizontal
- R26: renamed from R11; footprint Resistor_THT:R_Axial_DIN0207_L6.3mm_D2.5mm_P10.16mm_Horizontal -> cynthia:R_Axial_DIN0207_L6.3mm_D2.5mm_P10.16mm_Horizontal
- R27: renamed from R6; footprint Resistor_THT:R_Axial_DIN0207_L6.3mm_D2.5mm_P10.16mm_Horizontal -> cynthia:R_Axial_DIN0207_L6.3mm_D2.5mm_P10.16mm_Horizontal
- R28: renamed from R31; footprint Resistor_THT:R_Axial_DIN0207_L6.3mm_D2.5mm_P10.16mm_Horizontal -> cynthia:R_Axial_DIN0207_L6.3mm_D2.5mm_P10.16mm_Horizontal
- R29: renamed from R4; footprint Resistor_THT:R_Axial_DIN0207_L6.3mm_D2.5mm_P10.16mm_Horizontal -> cynthia:R_Axial_DIN0207_L6.3mm_D2.5mm_P10.16mm_Horizontal
- R3: renamed from R48; footprint Resistor_THT:R_Axial_DIN0207_L6.3mm_D2.5mm_P10.16mm_Horizontal -> cynthia:R_Axial_DIN0207_L6.3mm_D2.5mm_P10.16mm_Horizontal
- R30: renamed from R29; footprint Resistor_THT:R_Axial_DIN0207_L6.3mm_D2.5mm_P10.16mm_Horizontal -> cynthia:R_Axial_DIN0207_L6.3mm_D2.5mm_P10.16mm_Horizontal
- R31: renamed from R30; footprint Resistor_THT:R_Axial_DIN0207_L6.3mm_D2.5mm_P10.16mm_Horizontal -> cynthia:R_Axial_DIN0207_L6.3mm_D2.5mm_P10.16mm_Horizontal
- R32: renamed from R5; footprint Resistor_THT:R_Axial_DIN0207_L6.3mm_D2.5mm_P10.16mm_Horizontal -> cynthia:R_Axial_DIN0207_L6.3mm_D2.5mm_P10.16mm_Horizontal
- R33: renamed from R22; footprint Resistor_THT:R_Axial_DIN0207_L6.3mm_D2.5mm_P10.16mm_Horizontal -> cynthia:R_Axial_DIN0207_L6.3mm_D2.5mm_P10.16mm_Horizontal
- R34: renamed from R32; footprint Resistor_THT:R_Axial_DIN0207_L6.3mm_D2.5mm_P10.16mm_Horizontal -> cynthia:R_Axial_DIN0207_L6.3mm_D2.5mm_P10.16mm_Horizontal
- R35: renamed from R12; footprint Resistor_THT:R_Axial_DIN0207_L6.3mm_D2.5mm_P10.16mm_Horizontal -> cynthia:R_Axial_DIN0207_L6.3mm_D2.5mm_P10.16mm_Horizontal
- R36: renamed from R13; footprint Resistor_THT:R_Axial_DIN0207_L6.3mm_D2.5mm_P10.16mm_Horizontal -> cynthia:R_Axial_DIN0207_L6.3mm_D2.5mm_P10.16mm_Horizontal
- R37: renamed from R33; footprint Resistor_THT:R_Axial_DIN0207_L6.3mm_D2.5mm_P10.16mm_Horizontal -> cynthia:R_Axial_DIN0207_L6.3mm_D2.5mm_P10.16mm_Horizontal
- R38: renamed from R14; footprint Resistor_THT:R_Axial_DIN0207_L6.3mm_D2.5mm_P10.16mm_Horizontal -> cynthia:R_Axial_DIN0207_L6.3mm_D2.5mm_P10.16mm_Horizontal
- R39: renamed from R15; footprint Resistor_THT:R_Axial_DIN0207_L6.3mm_D2.5mm_P10.16mm_Horizontal -> cynthia:R_Axial_DIN0207_L6.3mm_D2.5mm_P10.16mm_Horizontal
- R4: renamed from R43; footprint Resistor_THT:R_Axial_DIN0207_L6.3mm_D2.5mm_P10.16mm_Horizontal -> cynthia:R_Axial_DIN0207_L6.3mm_D2.5mm_P10.16mm_Horizontal
- R40: renamed from R34; footprint Resistor_THT:R_Axial_DIN0207_L6.3mm_D2.5mm_P10.16mm_Horizontal -> cynthia:R_Axial_DIN0207_L6.3mm_D2.5mm_P10.16mm_Horizontal
- R41: renamed from R16; footprint Resistor_THT:R_Axial_DIN0207_L6.3mm_D2.5mm_P10.16mm_Horizontal -> cynthia:R_Axial_DIN0207_L6.3mm_D2.5mm_P10.16mm_Horizontal
- R42: renamed from R35; footprint Resistor_THT:R_Axial_DIN0207_L6.3mm_D2.5mm_P10.16mm_Horizontal -> cynthia:R_Axial_DIN0207_L6.3mm_D2.5mm_P10.16mm_Horizontal
- R44: renamed from R17; footprint Resistor_THT:R_Axial_DIN0207_L6.3mm_D2.5mm_P10.16mm_Horizontal -> cynthia:R_Axial_DIN0207_L6.3mm_D2.5mm_P10.16mm_Horizontal
- R45: renamed from R36; footprint Resistor_THT:R_Axial_DIN0207_L6.3mm_D2.5mm_P10.16mm_Horizontal -> cynthia:R_Axial_DIN0207_L6.3mm_D2.5mm_P10.16mm_Horizontal
- R46: renamed from R18; footprint Resistor_THT:R_Axial_DIN0207_L6.3mm_D2.5mm_P10.16mm_Horizontal -> cynthia:R_Axial_DIN0207_L6.3mm_D2.5mm_P10.16mm_Horizontal
- R47: renamed from R19; footprint Resistor_THT:R_Axial_DIN0207_L6.3mm_D2.5mm_P10.16mm_Horizontal -> cynthia:R_Axial_DIN0207_L6.3mm_D2.5mm_P10.16mm_Horizontal
- R48: renamed from R38; footprint Resistor_THT:R_Axial_DIN0207_L6.3mm_D2.5mm_P10.16mm_Horizontal -> cynthia:R_Axial_DIN0207_L6.3mm_D2.5mm_P10.16mm_Horizontal
- R49: renamed from R40; footprint Resistor_THT:R_Axial_DIN0207_L6.3mm_D2.5mm_P10.16mm_Horizontal -> cynthia:R_Axial_DIN0207_L6.3mm_D2.5mm_P10.16mm_Horizontal
- R5: renamed from R44; footprint Resistor_THT:R_Axial_DIN0207_L6.3mm_D2.5mm_P10.16mm_Horizontal -> cynthia:R_Axial_DIN0207_L6.3mm_D2.5mm_P10.16mm_Horizontal
- R50: renamed from R20; footprint Resistor_THT:R_Axial_DIN0207_L6.3mm_D2.5mm_P10.16mm_Horizontal -> cynthia:R_Axial_DIN0207_L6.3mm_D2.5mm_P10.16mm_Horizontal
- R51: renamed from R41; footprint Resistor_THT:R_Axial_DIN0207_L6.3mm_D2.5mm_P10.16mm_Horizontal -> cynthia:R_Axial_DIN0207_L6.3mm_D2.5mm_P10.16mm_Horizontal
- R52: renamed from R39; footprint Resistor_THT:R_Axial_DIN0207_L6.3mm_D2.5mm_P10.16mm_Horizontal -> cynthia:R_Axial_DIN0207_L6.3mm_D2.5mm_P10.16mm_Horizontal
- R8: renamed from R45; footprint Resistor_THT:R_Axial_DIN0207_L6.3mm_D2.5mm_P10.16mm_Horizontal -> cynthia:R_Axial_DIN0207_L6.3mm_D2.5mm_P10.16mm_Horizontal
- R9: renamed from R49; footprint Resistor_THT:R_Axial_DIN0207_L6.3mm_D2.5mm_P10.16mm_Horizontal -> cynthia:R_Axial_DIN0207_L6.3mm_D2.5mm_P10.16mm_Horizontal
- RV6: renamed from RV7; footprint Potentiometer_THT:Potentiometer_Bourns_3386W_Horizontal -> cynthia:trimmer
- renumbered C17 to C10, C7 to C16, C9 to C4, C12 to C5, C13 to C6, C14 to C7, C15 to C8, C16 to C9, D13 to D1, D3 to D10, D7 to D11, D9 to D12, D10 to D13, D8 to D14, D2 to D15, D11 to D16, D12 to D2, D14 to D5, D5 to D6, D1 to D7, D6 to D8, D4 to D9, Q12 to Q1, Q5 to Q10, Q6 to Q11, Q10 to Q12, Q11 to Q13, Q13 to Q2, Q2 to Q3, Q7 to Q4, Q3 to Q5, Q4 to Q6, Q9 to Q7, Q1 to Q8, Q8 to Q9, U2 to U1, U1 to U2
Connections:
- net +12V: now also D17.1 (K), D3.1 (K), J2.12 (Pin_12)
- net -12V: now also R15.1
- net GND: now also D18.2 (A), D4.2 (A), J2.11 (Pin_11), J3.S, J3.TN, J4.S, J4.TN, J5.S, J5.TN, J6.S, J6.TN, J7.S, J7.TN, R1.1; no longer R15.1
- net accent cv: now also J4.T, R6.1; no longer Q1.2 (B)
- net decay cv: now also J6.T, R43.1; no longer Q13.2 (B)
- net gate in: now also J3.T, R1.2
- net out: now also J7.T
- net pulse: now also J2.16 (Pin_16)
- net sine: now also J2.18 (Pin_18)
- net tune 1: now also J2.6 (Pin_6)
- net tune 2: now also J2.5 (Pin_5)
- net tune cv: now also J2.1 (Pin_1), J5.T
- net io fm on/off pin 1: now reaches C13.1, R27.2, U2.1, U2.6 (-)
- net io fm on/off pin 1: now also J2.20 (Pin_20)
- net io tune lvl pin 2: now reaches D7.2 (A)
- net io tune lvl pin 2: now also J2.2 (Pin_2)
- net io decay pin 2: now reaches R49.2, R51.2
- net io decay pin 2: now also J2.14 (Pin_14); no longer Q13.3 (E)
- net io tune decay 1: now reaches C4.1, D1.1 (K), D5.2 (A)
- net io tune decay 1: now also J2.3 (Pin_3)
- net io sine/pulse pin 2: now reaches R37.1
- net io sine/pulse pin 2: now also J2.17 (Pin_17)
- net io decay pin 1: now reaches C16.1, D16.1 (K), R42.1, R45.1
- net io decay pin 1: now also J2.15 (Pin_15)
- net io tune 1 pin 3: now reaches Q3.3 (E)
- net io tune 1 pin 3: now also J2.7 (Pin_7)
- net io tune 2 pin 2: now reaches R18.1
- net io tune 2 pin 2: now also J2.8 (Pin_8)
- net at R49.1: now also Q13.3 (E)
- net io tune 2 pin 3: now reaches Q5.3 (E)
- net io tune 2 pin 3: now also J2.9 (Pin_9)
- net io fm on/off pin 2: now reaches R33.1
- net io fm on/off pin 2: now also J2.19 (Pin_19)
- net io tune depth 1: now reaches R9.2
- net io tune depth 1: now also J2.4 (Pin_4)
- new net: D3.2 (A), D4.1 (K), Q1.2 (B), R6.2
- new net: D17.2 (A), D18.1 (K), Q13.2 (B), R43.2
- no-connect marks 0 -> 12
Other:
- moved on the sheet: D7, Q13, Q5, R15, R18, R49, R51
