File: 11_fm_drum/11_fm_drum_io/11_fm_drum_io.kicad_sch (KiCad schematic)
At the start: 0 parts

Commit message: updated 11 io
Parts:
- added J1: Conn_02x10_Counter_Clockwise, Connector_PinHeader_2.54mm:PinHeader_2x10_P2.54mm_Vertical, symbol Connector_Generic:Conn_02x10_Counter_Clockwise
- added R1: 33k, cynthia:R_Axial_DIN0207_L6.3mm_D2.5mm_P10.16mm_Horizontal, symbol Device:R
- added R2: 1k, cynthia:R_Axial_DIN0207_L6.3mm_D2.5mm_P10.16mm_Horizontal, symbol Device:R
- added RV1, RV4, RV5: 100k, cynthia:potientiometer, symbol Device:R_Potentiometer
- added RV2: 1M, cynthia:potientiometer, symbol Device:R_Potentiometer
- added RV3: 250k, cynthia:potientiometer, symbol Device:R_Potentiometer
- added RV6: 500k, cynthia:potientiometer, symbol Device:R_Potentiometer
- added SW1, SW2: SW_SPDT, cynthia:switch, symbol Switch:SW_SPDT
Connections:
- new net: R2.2, RV3.2, RV3.3
- new net: R1.1, RV5.3
- new net +12V: J1.12 (Pin_12), R1.2, RV4.1
- new net GND: J1.11 (Pin_11), R2.1, RV1.3, SW1.3 (C)
- new net io decay pin 1: J1.15 (Pin_15), RV6.1
- new net io decay pin 2: J1.14 (Pin_14), RV6.2, RV6.3
- new net io fm on/off pin 1: J1.20 (Pin_20), SW1.1 (A)
- new net io fm on/off pin 2: J1.19 (Pin_19), SW1.2 (B)
- new net io sine/pulse pin 1: J1.18 (Pin_18), SW2.1 (A)
- new net io sine/pulse pin 2: J1.17 (Pin_17), SW2.2 (B)
- new net io sine/pulse pin 3: J1.16 (Pin_16), SW2.3 (C)
- new net io tune 1 pin 2: J1.6 (Pin_6), RV4.2
- new net io tune 1 pin 3: J1.7 (Pin_7), RV4.3
- new net io tune 2 pin 2: J1.8 (Pin_8), RV5.2
- new net io tune 2 pin 3: J1.9 (Pin_9), RV5.1
- new net io tune decay 1: J1.3 (Pin_3), RV3.1
- new net io tune depth 1: J1.4 (Pin_4), RV2.1, RV2.2
- new net io tune depth 2: J1.5 (Pin_5), RV2.3
- new net io tune lvl pin 1: J1.1 (Pin_1), RV1.1
- new net io tune lvl pin 2: J1.2 (Pin_2), RV1.2
- no-connect marks 0 -> 2
