File: 11_fm_drum/11_fm_drum/11_fm_drum.kicad_pcb (KiCad board)
At the start: 2 copper layers, 80 x 100 mm, 123 parts, among them J1 Conn_02x05_Odd_Even, J2 Conn_01x06, Q1 BC558, Q10 BC548, Q11 BC548, Q12 BC548, Q13 BC558, Q2 BC548, Q3 BC558, Q4 BC548, Q5 BC558, Q6 BC548, Q7 BC558, Q8 BC548, Q9 BC548, SW1 SW_SPDT, SW2 SW_SPDT, U1 TL072, U2 TL074

Commit message: ordered 11
Parts:
- added H1: MountingHole, MountingHole:MountingHole_3.2mm_M3, F.Cu at (124.0, 26.0)
- added H2: MountingHole, MountingHole:MountingHole_3.2mm_M3, F.Cu at (124.0, 116.0)
- C1: value 10nF -> 103
- C11: value 5.6nF -> 562
- C12, C14: value 470pF -> 471; footprint Capacitor_THT:C_Rect_L7.2mm_W3.5mm_P5.00mm_FKS2_FKP2_MKS2_MKP2 -> Capacitor_THT:C_Rect_L7.2mm_W2.5mm_P5.00mm_FKS2_FKP2_MKS2_MKP2
- C13: value 2.2nF -> 222
- C15: value 15nF -> 153
- C16: value 1uF -> 105
- C17: value 330pF -> 331
- C4: value 470nF -> 474
- C5, C6, C7: value 100nF -> 104
- moved R10 6.80 mm to (141.9, 114.1)
- moved R8 6.80 mm to (141.9, 117.1)
- moved R51 6.54 mm to (144.3, 117.3)
- moved R52 6.54 mm to (144.2, 113.7)
- moved RV7 5.91 mm to (186.2, 117.1)
- moved R43 5.85 mm to (159.8, 117.1)
- moved R49 5.85 mm to (159.8, 114.1)
- moved Q13 5.63 mm to (178.5, 114.6)
- moved C6 5.57 mm to (157.0, 30.0)
- moved C2 4.89 mm to (164.2, 26.0)
- moved C3 4.89 mm to (173.0, 26.0)
- moved C5 4.24 mm to (154.0, 25.0)
- moved C1 2.89 mm to (123.4, 94.3)
- moved RV2 2.27 mm to (192.5, 109.7)
- moved C4 1.04 mm to (136.1, 85.3)
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Routing:
- net +12V: track 247.1 -> 267.6 mm, vias 1 -> 0
- net Net-(D16-K): track 48.5 -> 68.4 mm, vias 0 -> 1
- net -12V: track 147.7 -> 163.6 mm, vias 2 -> 1
- net trigger: track 161.2 -> 151.4 mm, vias 2 -> 1
- net GND: track 396.0 -> 405.1 mm
- net Net-(Q9-E): track 49.1 -> 58.2 mm
- net Net-(D11-K): track 35.3 -> 43.2 mm, vias 1 -> 0
- net Net-(Q2-B): track 34.9 -> 27.4 mm
- net out: track 50.5 -> 43.8 mm
- net tune 2: track 90.9 -> 84.2 mm
- net decay cv: track 50.9 -> 45.2 mm
- net square 2: track 100.9 -> 95.4 mm, vias 2 -> 1
- net Net-(R48-Pad2): track 46.0 -> 40.7 mm
- net Net-(Q9-B): track 61.7 -> 56.4 mm, vias 2 -> 1
- net Net-(R9-Pad2): track 100.3 -> 95.4 mm
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
Commit message: fixed details on pcb for 11
Parts:
- C8: value 100nF -> 104
Changed lines of the file:
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@@
 		(property "Value" "BC558"
 			(at 1.27 2.79 90)
-			(layer "F.Fab")
+			(layer "F.SilkS")
 			(effects
 				(font
@@
 			)
 		)
-		(property "Value" "100nF"
-			(at 2.5 2.5 90)
-			(layer "F.Fab")
-			(hide yes)
-			(effects
-				(font
+		(property "Value" "104"
+			(at 2.5 0.038456 90)
+			(layer "F.SilkS")
+			(effects
+				(font
