File: 11_fm_drum/11_fm_drum/11_fm_drum.kicad_sch (KiCad schematic)
At the start: 108 parts, among them J1 Conn_02x05_Odd_Even, J2 Conn_02x10_Counter_Clockwise, J3 Gate IN, J4 Acceent CV, J5 Tune CV, J6 Decay CV, J7 Out, Q1 BC558, Q10 BC548, Q11 BC548, Q12 BC548, Q13 BC558, Q2 BC548, Q3 BC558, Q4 BC548, Q5 BC558, Q6 BC548, Q7 BC558, Q8 BC548, Q9 BC548, U1 TL072, U2 TL074

Commit message: removed io from 11
Parts:
- removed J2: Conn_02x10_Counter_Clockwise, Connector_PinSocket_2.54mm:PinSocket_2x10_P2.54mm_Vertical, symbol Connector_Generic:Conn_02x10_Counter_Clockwise
- removed J3: Gate IN, cynthia:6.25mm Jack Stereo Switched, symbol cynthia:6.35_mm_jack_socket_stereo_switched
- removed J4: Acceent CV, cynthia:6.25mm Jack Stereo Switched, symbol cynthia:6.35_mm_jack_socket_stereo_switched
- removed J5: Tune CV, cynthia:6.25mm Jack Stereo Switched, symbol cynthia:6.35_mm_jack_socket_stereo_switched
- removed J6: Decay CV, cynthia:6.25mm Jack Stereo Switched, symbol cynthia:6.35_mm_jack_socket_stereo_switched
- removed J7: Out, cynthia:6.25mm Jack Stereo Switched, symbol cynthia:6.35_mm_jack_socket_stereo_switched
- added J2: Conn_01x06, Connector_PinHeader_2.54mm:PinHeader_1x06_P2.54mm_Vertical, symbol Connector_Generic:Conn_01x06
- added R17: 33k, cynthia:R_Axial_DIN0207_L6.3mm_D2.5mm_P10.16mm_Horizontal, symbol Device:R
- added R7: 1k, cynthia:R_Axial_DIN0207_L6.3mm_D2.5mm_P10.16mm_Horizontal, symbol Device:R
- added RV1, RV4, RV5: 100k, Connector_PinHeader_2.54mm:PinHeader_1x03_P2.54mm_Vertical, symbol Device:R_Potentiometer
- added RV2: 1M, Connector_PinHeader_2.54mm:PinHeader_1x03_P2.54mm_Vertical, symbol Device:R_Potentiometer
- added RV3: 250k, Connector_PinHeader_2.54mm:PinHeader_1x03_P2.54mm_Vertical, symbol Device:R_Potentiometer
- added RV7: 500k, Connector_PinHeader_2.54mm:PinHeader_1x03_P2.54mm_Vertical, symbol Device:R_Potentiometer
- added SW1, SW2: SW_SPDT, Connector_PinHeader_2.54mm:PinHeader_1x03_P2.54mm_Vertical, symbol Switch:SW_SPDT
- added TP1, TP10, TP2, TP3, TP4, TP5, TP6, TP7, TP8, TP9: TestPoint, TestPoint:TestPoint_Pad_1.0x1.0mm, symbol Connector:TestPoint
Connections:
- net +12V: now also R17.1, RV4.3
- net GND: now also U1.3 (+), J2.6 (Pin_6), R7.1, RV1.3, SW1.3 (C); no longer U1.5 (+)
- net accent cv: now also J2.3 (Pin_3)
- net accented trigger: now also TP10.1
- net decay cv: now also J2.4 (Pin_4)
- net gate in: now also J2.1 (Pin_1)
- net out: now also J2.5 (Pin_5)
- net pulse: now also SW2.3 (C)
- net sine: now also SW2.1 (A), TP5.1
- net square 1: now also TP3.1
- net square 2: now also TP8.1
- net triangle 2: now also TP4.1
- net trigger: now also U1.7; no longer U1.1
- net tune 1: now also RV4.2
- net tune 2: now also RV2.3
- net tune cv: now also J2.2 (Pin_2), RV1.1
- net at C15.1, R34.1: now also TP6.1
- net at C1.2, D2.1 (K), R4.2: now also U1.5 (+); no longer U1.3 (+)
- net at R2.2, R5.1: now also U1.6 (-); no longer U1.2 (-)
- net at C12.2, Q7.1 (C), R25.2: now also TP9.1
- net at Q12.3 (E), R48.1, RV6.1: now also U1.2 (-); no longer U1.6 (-)
- net at R48.2, R52.1: now also U1.1; no longer U1.7
- net io decay pin 1: no longer names the net of C16.1, D16.1 (K), R42.1, R45.1
- net io decay pin 1: now also RV7.1, TP7.1
- net io decay pin 2: no longer names the net of R49.2, R51.2
- net io decay pin 2: now also RV7.2, RV7.3
- net io fm on/off pin 1: no longer names the net of C13.1, R27.2, U2.1, U2.6 (-)
- net io fm on/off pin 1: now also SW1.1 (A), TP2.1
- net io fm on/off pin 2: no longer names the net of R33.1
- net io fm on/off pin 2: now also SW1.2 (B)
- net io sine/pulse pin 2: no longer names the net of R37.1
- net io sine/pulse pin 2: now also SW2.2 (B)
- net io tune 1 pin 3: no longer names the net of Q3.3 (E)
- net io tune 1 pin 3: now also RV4.1
- net io tune 2 pin 2: no longer names the net of R18.1
- net io tune 2 pin 2: now also RV5.2
- net io tune 2 pin 3: no longer names the net of Q5.3 (E)
- net io tune 2 pin 3: now also RV5.1
- net io tune decay 1: no longer names the net of C4.1, D1.1 (K), D5.2 (A)
- net io tune decay 1: now also RV3.1, TP1.1
- net io tune depth 1: no longer names the net of R9.2
- net io tune depth 1: now also RV2.1, RV2.2
- net io tune lvl pin 2: no longer names the net of D7.2 (A)
- net io tune lvl pin 2: now also RV1.2
- new net: R7.2, RV3.2, RV3.3
- new net: R17.2, RV5.3
- no-connect marks 12 -> 0
Other:
- moved on the sheet: D7, Q5, R18

Commit message: ordered 11
Parts:
- added H1, H2: MountingHole, MountingHole:MountingHole_3.2mm_M3, symbol Mechanical:MountingHole
- C12, C14: footprint Capacitor_THT:C_Rect_L7.2mm_W3.5mm_P5.00mm_FKS2_FKP2_MKS2_MKP2 -> Capacitor_THT:C_Rect_L7.2mm_W2.5mm_P5.00mm_FKS2_FKP2_MKS2_MKP2
Changed lines of the file:
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@@
 			)
 		)
-		(property "Footprint" "Capacitor_THT:C_Rect_L7.2mm_W3.5mm_P5.00mm_FKS2_FKP2_MKS2_MKP2"
+		(property "Footprint" "Capacitor_THT:C_Rect_L7.2mm_W2.5mm_P5.00mm_FKS2_FKP2_MKS2_MKP2"
 			(at 265.43 95.5548 0)
 			(effects
@@
 			)
 		)
-		(property "Footprint" "Capacitor_THT:C_Rect_L7.2mm_W3.5mm_P5.00mm_FKS2_FKP2_MKS2_MKP2"
+		(property "Footprint" "Capacitor_THT:C_Rect_L7.2mm_W2.5mm_P5.00mm_FKS2_FKP2_MKS2_MKP2"
 			(at 254 95.5548 0)
 			(effects
@@
 	)
 	(symbol
+		(lib_id "Mechanical:MountingHole")
+		(at 182.88 152.4 0)
+		(unit 1)
+		(exclude_from_sim no)
+		(in_bom no)
+		(on_board yes)
+		(dnp no)
+		(fields_autoplaced yes)
+		(property "Reference" "H2"
+			(at 185.42 151.1299 0)
+			(effects
+				(font
+					(size 1.27 1.27)
+				)
+				(justify left)
+			)
+		)
+		(property "Value" "MountingHole"
+			(at 185.42 153.6699 0)
+			(effects
+				(font
+					(size 1.27 1.27)
+				)
+				(justify left)
+			)
+		)
+		(property "Footprint" "MountingHole:MountingHole_3.2mm_M3"
+			(at 182.88 152.4 0)
+			(effects
+				(font
+					(size 1.27 1.27)
+				)
+				(hide yes)
+			)
+		)
+		(property "Datasheet" "~"
+			(at 182.88 152.4 0)
+			(effects
+				(font
+					(size 1.27 1.27)
+				)
+				(hide yes)
+			)
+		)
+		(property "Description" "Mounting Hole without connection"
+			(at 182.88 152.4 0)
+			(effects
+				(font
+					(size 1.27 1.27)
+				)
+				(hide yes)
+			)
+		)
+		(instances
+			(project "11_fm_drum"
+				(path "/41198931-f787-4e52-811f-ac8bc7c779e9"
+					(reference "H2")
+					(unit 1)
+				)
+			)
+		)
+	)
+	(symbol
 		(lib_id "Device:R")
 		(at 381 58.42 90)
@@
 					(unit 1)
 				)
+			)
+		)
+	)
+	(symbol
+		(lib_id "Mechanical:MountingHole")
+		(at 182.88 146.05 0)
+		(unit 1)
+		(exclude_from_sim no)
+		(in_bom no)
+		(on_board yes)
+		(dnp no)
+		(fields_autoplaced yes)
+		(property "Reference" "H1"
+			(at 185.42 144.7799 0)
+			(effects
+				(font
+					(size 1.27 1.27)
+				)
+				(justify left)
+			)
+		)
+		(property "Value" "MountingHole"
+			(at 185.42 147.3199 0)
+			(effects
+				(font
+					(size 1.27 1.27)
+				)
+				(justify left)
+			)
+		)
+		(property "Footprint" "MountingHole:MountingHole_3.2mm_M3"
+			(at 182.88 146.05 0)
+			(effects
+				(font
+					(size 1.27 1.27)
+				)
+				(hide yes)
+			)
+		)
+		(property "Datasheet" "~"
+			(at 182.88 146.05 0)
+			(effects
+				(font
+					(size 1.27 1.27)
+				)
+				(hide yes)
+			)
+		)
+		(property "Description" "Mounting Hole without connection"
+			(at 182.88 146.05 0)
+			(effects
+				(font
+					(size 1.27 1.27)
+				)
+				(hide yes)
+			)
+		)
+		(instances
+			(project ""
+				(path "/41198931-f787-4e52-811f-ac8bc7c779e9"
+					(reference "H1")
+					(unit 1)
+				)

Commit message: fixed details on pcb for 11
Parts:
- R10: value 3.3 -> 3.3k
Changed lines of the file:
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@@
 			)
 		)
-		(property "Value" "3.3"
+		(property "Value" "3.3k"
 			(at 85.09 50.8 90)
 			(effects
