File: 03_env_pluck/schematics/03_env_vca.kicad_sch (KiCad schematic)
At the start: 45 parts, among them J1 gate in 1, J3 Eurorack, J4 signal in, J5 Env out 1, J7 Signal out, Q1 BC847, Q2 BC847, SW1 Pluck / AD 1, U2 LM358, U3 TL072

Commit message: updated references
Parts:
- renumbered C3 to C2, C4 to C3, C5 to C4, C7 to C5, C9 to C6, C10 to C7, D2 to D1, D5 to D2, D6 to D3, J4 to J2, J7 to J4, R15 to R1, R22 to R10, R23 to R11, R6 to R12, R9 to R13, R10 to R14, R24 to R15, R25 to R16, R26 to R17, R12 to R18, R27 to R19, R16 to R2, R28 to R20, R29 to R21, R14 to R22, R1 to R3, R17 to R4, R18 to R5, R3 to R6, R19 to R7, R20 to R8, R21 to R9, RV5 to RV1, RV3 to RV2, RV4 to RV3, U3 to U1
Connections:
- net Env: now reaches R1.1, R22.1, U2.1, U2.2 (-)
Other:
- moved on the sheet: J2, J4, Q1, Q2, R1, R10, R11, R15, R16, R17, R19, R2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

Commit message: cleanup
Parts:
- J1: value gate in 1 -> gate in
- J5: value Env out 1 -> env out
- renumbered R15 to R12, R16 to R13, R17 to R14, R12 to R15, R13 to R16, R14 to R17, R19 to R18, R20 to R19, R18 to R20, R4 to R3, R5 to R4, R3 to R5, R7 to R6, R8 to R7, R6 to R8
Connections:
- net Env renamed env
Other:
- moved on the sheet: C1, C5, D1, D2, D3, J1, J2, J4, J5, Q1, Q2, R1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
