File: 03_env_pluck/schematics/03_env_vca.kicad_sch (KiCad schematic)
At the start: 45 parts, among them J1 gate in, J2 signal in, J3 Eurorack, J4 Signal out, J5 env out, Q1 BC847, Q2 BC847, SW1 Pluck / AD 1, U1 TL072, U2 LM358

Commit message: 3d modules for 03
Parts:
- J4, J5: footprint cynthia:3.5mm jack mono -> cynthia:3.5mm jack mono switched; symbol Connector_Audio:AudioJack2 -> Connector_Audio:AudioJack2_SwitchT
Connections:
- no-connect marks 0 -> 2
Changed lines of the file:
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@@
 		(color 0 0 0 0)
 	)
+	(no_connect
+		(at 182.88 31.75)
+	)
+	(no_connect
+		(at 139.7 81.28)
+	)
 	(wire
 		(pts
@@
 	)
 	(symbol
-		(lib_id "Connector_Audio:AudioJack2")
+		(lib_id "Connector_Audio:AudioJack2_SwitchT")
 		(at 187.96 34.29 180)
 		(unit 1)
@@
 			)
 		)
-		(property "Footprint" "cynthia:3.5mm jack mono"
+		(property "Footprint" "cynthia:3.5mm jack mono switched"
 			(at 187.96 34.29 0)
 			(hide yes)
@@
 			)
 		)
-		(property "Description" "Audio Jack, 2 Poles (Mono / TS)"
+		(property "Description" "Audio Jack, 2 Poles (Mono / TS), Switched T Pole (Normalling)"
 			(at 187.96 34.29 0)
 			(hide yes)
@@
 		(pin "T"
 		)
+		(pin "TN"
+		)
 		(instances
 			(project "03_env_vca"
@@
 	)
 	(symbol
-		(lib_id "Connector_Audio:AudioJack2")
+		(lib_id "Connector_Audio:AudioJack2_SwitchT")
 		(at 144.78 83.82 180)
 		(unit 1)
@@
 			)
 		)
-		(property "Footprint" "cynthia:3.5mm jack mono"
+		(property "Footprint" "cynthia:3.5mm jack mono switched"
 			(at 144.78 83.82 0)
 			(hide yes)
@@
 			)
 		)
-		(property "Description" "Audio Jack, 2 Poles (Mono / TS)"
+		(property "Description" "Audio Jack, 2 Poles (Mono / TS), Switched T Pole (Normalling)"
 			(at 144.78 83.82 0)
 			(hide yes)
@@
 		(pin "T"
 		)
+		(pin "TN"
+		)
 		(instances
