File: 13_dual_env/schematics/13_dual_env.kicad_pcb (KiCad board)
At the start: 2 copper layers, 20 x 109 mm, 42 parts, among them J1 gate in, J2 gate in, J3 Eurorack, J5 env out, J6 env out, SW1 Pluck / AD 1, SW2 Pluck / AD 1, U1 TL072, U2 LM358

Commit message: added PCB for 13
Parts:
- removed C1: 47nF, Capacitor_SMD:C_0805_2012Metric_Pad1.18x1.45mm_HandSolder
- removed C4: 100nF, Capacitor_SMD:C_0805_2012Metric_Pad1.18x1.45mm_HandSolder
- removed J2: gate in, cynthia:3.5mm jack mono switched
- removed R8: 100k, Resistor_SMD:R_0805_2012Metric_Pad1.20x1.40mm_HandSolder
- removed RV4, RV5: 1M, cynthia:potientiometer
- added C10: 100nF, Capacitor_SMD:C_0805_2012Metric_Pad1.18x1.45mm_HandSolder, F.Cu at (7.50, 52.0)
- added C11: 100nF, Capacitor_SMD:C_0805_2012Metric_Pad1.18x1.45mm_HandSolder, F.Cu at (10.5, 64.0)
- added D7: 1N4148, Diode_SMD:D_0805_2012Metric_Pad1.15x1.40mm_HandSolder, F.Cu at (8.00, 78.0)
- added D8: LED, LED_THT:LED_D5.0mm, B.Cu at (-1.77, 87.0)
- added Q1: BC848, Package_TO_SOT_SMD:SOT-23, F.Cu at (8.00, 75.0)
- added Q2: BC858, Package_TO_SOT_SMD:SOT-23, F.Cu at (19.5, 61.5)
- added Q3: BC848, Package_TO_SOT_SMD:SOT-23, F.Cu at (8.00, 93.0)
- added Q4: BC858, Package_TO_SOT_SMD:SOT-23, F.Cu at (-2.50, 92.5)
- added R25: 22k, Resistor_SMD:R_0805_2012Metric_Pad1.20x1.40mm_HandSolder, F.Cu at (18.0, 57.5)
- added R26: 100k, Resistor_SMD:R_0805_2012Metric_Pad1.20x1.40mm_HandSolder, F.Cu at (10.5, 21.5)
- added R27: 100k, Resistor_SMD:R_0805_2012Metric_Pad1.20x1.40mm_HandSolder, F.Cu at (8.00, 7.50)
- added R28: 1k, Resistor_SMD:R_0805_2012Metric_Pad1.20x1.40mm_HandSolder, F.Cu at (17.5, 97.0)
- added R7: 100k, Resistor_SMD:R_0805_2012Metric_Pad1.20x1.40mm_HandSolder, F.Cu at (10.5, 17.5)
- added SW3: ~, cynthia:switch_dpdt, B.Cu at (17.0, 70.0)
- added SW4: Gate/Loop, cynthia:switch_spdt, B.Cu at (17.0, 24.5)
- C5: footprint Capacitor_SMD:C_0805_2012Metric_Pad1.18x1.45mm_HandSolder -> Capacitor_THT:C_Rect_L7.0mm_W6.5mm_P5.00mm
- C8: value 47nF -> 100nF
- C9: value 1uF -> 100nF
- D4: value 1N4148 -> LED; footprint Diode_SMD:D_0805_2012Metric_Pad1.15x1.40mm_HandSolder -> LED_THT:LED_D5.0mm; moved to B.Cu
- J1: value gate in -> gate in 1; moved to B.Cu
- J3: footprint Connector_PinHeader_2.54mm:PinHeader_2x05_P2.54mm_Vertical -> cynthia:Eurorack Header
- J5: value env out -> env out 1; moved to B.Cu
- J6: value env out -> End of Cycle Out; moved to B.Cu
- R16: value 82k -> 100k
- R17: value 18k -> 22k
- R18: value 100k -> 33k
- R19: value 82k -> 8.2k
- R20, R23: value 560R -> 1k
- R21: value 18k -> 100k
- R24: value 1k -> 10k
- RV2, RV3: moved to B.Cu
- SW1: value Pluck / AD 1 -> Manual Gate; footprint cynthia:switch -> cynthia:push button; moved to B.Cu
- SW2: value Pluck / AD 1 -> Normal/Inverted; footprint cynthia:switch -> cynthia:switch_spdt; moved to B.Cu
- U1: value TL072 -> TL074; footprint Package_SO:SOIC-8_3.9x4.9mm_P1.27mm -> cynthia:SOIC-14_3.9x8.7mm_P1.27mm
- U2: value LM358 -> TL072; footprint Package_SO:SOIC-8_3.9x4.9mm_P1.27mm -> cynthia:SOIC-8_3.9x4.9mm_P1.27mm
- moved J6 80.3 mm to (17.0, 97.0), turned to 180 degrees
- moved RV2 77.7 mm to (17.0, 37.5), turned to 180 degrees
- moved SW2 76.7 mm to (17.0, 83.5), turned to 180 degrees
- moved J5 75.6 mm to (3.00, 97.0), turned to 180 degrees
- moved D5 73.4 mm to (13.0, 7.50)
- moved J1 73.1 mm to (17.0, 11.5), turned to 180 degrees
- moved C9 69.8 mm to (20.0, 57.5), turned to 90 degrees
- moved C8 69.0 mm to (11.0, 71.0), turned to 90 degrees
- moved D6 68.4 mm to (22.0, 57.5), turned to 90 degrees
- moved C5 67.6 mm to (15.0, 52.0)
- moved R22 67.4 mm to (2.50, 96.5)
- moved D4 64.7 mm to (5.22, 87.0)
- moved D2 63.8 mm to (14.5, 61.0)
- moved R23 59.0 mm to (3.00, 90.0)
- moved D3 57.8 mm to (7.50, 66.0), turned to 90 degrees
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Connections:
- C5 pad 1: Net-(U1A-+) -> Net-(D2-K)
- C8 pad 1: Net-(C8-Pad1) -> Net-(Q1-B)
- C8 pad 2: Net-(SW2-A) -> GND
- C9 pad 1: Net-(U1B-+) -> Net-(Q2-B)
- D3 pad 1: Net-(D2-A) -> Net-(D3-K)
- D3 pad 2: Net-(D3-A) -> Net-(D2-K)
- D4 pad 1: Net-(D4-K) -> GND
- D6 pad 1: Net-(D5-A) -> Net-(D6-K)
- J1 pad T: Net-(C1-Pad1) -> Net-(D5-A)
- R16 pad 1: Net-(U2A--) -> Net-(U1A--)
- R17 pad 1: unconnected-(R17-Pad1) -> GND
- R17 pad 2: Net-(U2A--) -> Net-(U1A--)
- R18 pad 1: GND -> Net-(Q1-B)
- R18 pad 2: Net-(D4-K) -> +12V
- R19 pad 1: Net-(U2B--) -> GND
- R19 pad 2: +12V -> Net-(Q1-B)
- R20 pad 1: Net-(R20-Pad1) -> Net-(U1B--)
- R20 pad 2: Net-(D2-A) -> Net-(R20-Pad2)
- R21 pad 1: unconnected-(R21-Pad1) -> Net-(U1D-+)
- R21 pad 2: Net-(U2B--) -> +12V
- R22 pad 1: env -> Net-(Q3-B)
- R23 pad 1: Net-(R23-Pad1) -> Net-(D4-A)
- R23 pad 2: Net-(D5-A) -> Net-(Q3-E)
- R24 pad 1: env -> Net-(Q2-B)
- R24 pad 2: Net-(J6-PadT) -> +12V
- R5 pad 1: Net-(C1-Pad1) -> Net-(D5-K)
- R5 pad 2: Net-(SW1-C) -> Net-(U1A-+)
- R6 pad 1: Net-(C8-Pad1) -> Net-(U2B--)
- R9 pad 1: GND -> Net-(SW2-A)
- R9 pad 2: Net-(SW2-A) -> Net-(U2B--)
- RV2 pad 1: Net-(D2-K) -> Net-(R20-Pad2)
- RV2 pad 2: Net-(U1A-+) -> Net-(D6-A)
- RV2 pad 3: Net-(U1A-+) -> Net-(D6-A)
- RV3 pad 1: Net-(D3-A) -> Net-(R20-Pad2)
- RV3 pad 2: Net-(U1A-+) -> Net-(D7-K)
- RV3 pad 3: Net-(U1A-+) -> Net-(D7-K)
- SW1 pad 1: Net-(SW1-A) -> Net-(D5-K)
- SW1 pad 2: Net-(D1-A) -> +12V
- SW2 pad 2: Net-(D4-A) -> Net-(Q3-B)
- U1 pad 1: env -> Net-(SW4-C)
- U1 pad 2: env -> Net-(U1A--)
- U1 pad 4: -12V -> +12V
- U1 pad 5: Net-(U1B-+) -> Net-(D1-K)
- U1 pad 6: env -> Net-(U1B--)
- U1 pad 7: env -> Net-(U1B--)
- U1 pad 8: +12V -> Net-(U1C--)
- U2 pad 1: Net-(R20-Pad1) -> Net-(SW2-A)
- U2 pad 2: Net-(U2A--) -> Net-(SW2-A)
- U2 pad 3: Net-(D1-K) -> Net-(D2-K)
- U2 pad 4: GND -> -12V
- U2 pad 5: Net-(D4-K) -> GND
- U2 pad 7: Net-(R23-Pad1) -> Net-(SW2-C)
Routing:
- net +12V: track 0.00 -> 168.9 mm, vias 0 -> 5
- net Net-(SW2-A): track 0.00 -> 115.4 mm
- net -12V: track 0.00 -> 103.7 mm, vias 0 -> 3
- net Net-(U1C--): track 0.00 -> 96.4 mm, vias 0 -> 2
- net Net-(SW2-C): track 0.00 -> 55.1 mm, vias 0 -> 2
- net Net-(D7-K): track 0.00 -> 53.6 mm
- net Net-(D6-A): track 0.00 -> 36.0 mm, vias 0 -> 1
- net Net-(SW4-A): track 0.00 -> 35.4 mm
- net Net-(Q3-B): track 0.00 -> 34.1 mm, vias 0 -> 2
- net Net-(R20-Pad2): track 0.00 -> 31.4 mm
- net Net-(D2-K): track 0.00 -> 26.0 mm
- net Net-(D3-K): track 0.00 -> 24.0 mm
- net GND: track 0.00 -> 23.3 mm, vias 0 -> 9
- net Net-(D1-A): track 0.00 -> 20.7 mm
- net Net-(SW4-C): track 0.00 -> 19.3 mm
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- added copper zone on B.Cu, net GND
Other:
- board size 20 x 109 mm -> 30 x 100 mm
