File: 13_dual_env/schematics/13_dual_env.kicad_sch (KiCad schematic)
At the start: 51 parts, among them J1 gate in 1, J3 Eurorack, J5 env out 1, J6 End of Cycle Out, Q1 BC848, Q2 BC858, Q3 BC848, Q4 BC858, SW1 Manual Gate, SW2 Normal/Inverted, SW4 Gate/Loop, U1 TL074, U2 TL072

Commit message: added PCB for 13
Parts:
- C5: footprint Capacitor_SMD:C_0805_2012Metric_Pad1.18x1.45mm_HandSolder -> Capacitor_THT:C_Rect_L7.0mm_W6.5mm_P5.00mm
- J3: footprint Connector_PinHeader_2.54mm:PinHeader_2x05_P2.54mm_Vertical -> cynthia:Eurorack Header
- SW1: footprint (none) -> cynthia:push button
- SW2, SW4: footprint cynthia:switch -> cynthia:switch_spdt
- SW3: footprint (none) -> cynthia:switch_dpdt
- U1: footprint (none) -> cynthia:SOIC-14_3.9x8.7mm_P1.27mm
- U2: footprint (none) -> cynthia:SOIC-8_3.9x4.9mm_P1.27mm
Connections:
- net at R9.1, SW2.1 (A), U2.1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: now also U1.13 (-); no longer U1.9 (-)
- net at R7.2, SW4.1 (A): now also U1.10 (+), U1.14; no longer U1.12 (+), U1.8
- net at R21.1, R26.2, R7.1: now also U1.12 (+); no longer U1.10 (+)
- new net: R28.1, U1.8, U1.9 (-)
