File: 15_oct_vca_mixer/15_oct_vca_mixer.kicad_pcb (KiCad board)
At the start: 2 copper layers, 70 x 100 mm, 149 parts, among them J1 Signal out, J10 CV in, J11 signal in, J12 CV in, J13 signal in, J2 CV in, J3 signal in, J4 CV in, J5 signal in, Q1 BC847BS, Q2 BC847BS, Q5 BC847BS, Q6 BC847BS, U1 TL072, U2 TL072, U3 TL072, U4 TL072, U5 TL072, U6 TL072, U7 TL072, U8 TL072, U9 TL072

Commit message: fine-tune 15 PCB
Parts:
- added TP1: TestPoint, TestPoint:TestPoint_Pad_2.0x2.0mm, B.Cu at (25.9, 61.5)
- added TP2: TestPoint, TestPoint:TestPoint_Pad_2.0x2.0mm, B.Cu at (62.0, 62.6)
- added TP3: TestPoint, TestPoint:TestPoint_Pad_2.0x2.0mm, B.Cu at (8.20, 61.5)
- added TP4: TestPoint, TestPoint:TestPoint_Pad_2.0x2.0mm, B.Cu at (44.0, 61.5)
- C1, C2: moved to F.Cu
- renumbered C20 to C10, C27 to C11, C28 to C12, C7 to C13, C8 to C14, C9 to C15, C10 to C16, C21 to C17, C22 to C18, C29 to C19, C30 to C20, C31 to C3, C32 to C4, C3 to C5, C4 to C6, C5 to C7, C6 to C8, C19 to C9, D7 to D4, D4 to D5, D8 to D6, J10 to J3, J3 to J4, J11 to J5, J4 to J6, J12 to J7, J5 to J8, J13 to J9, Q5 to Q2, Q2 to Q3, Q6 to Q4, R87 to R10, R8 to R11, R88 to R12, R10 to R13, R89 to R14, R11 to R15, R90 to R16, R9 to R17, R91 to R18, R12 to R19, R92 to R20, R13 to R21, R15 to R22, R93 to R23, R94 to R24, R14 to R25, R95 to R26, R16 to R27, R96 to R28, R17 to R29, R97 to R30, R18 to R31, R98 to R32, R19 to R33, R99 to R34, R20 to R35, R21 to R36, R100 to R37, R101 to R38, R22 to R39, R23 to R40, R102 to R41, R103 to R42, R24 to R43, R104 to R44, R25 to R45, R105 to R46, R26 to R47, R106 to R48, R27 to R49, R107 to R50, R28 to R51, R108 to R52, R29 to R53, R109 to R54, R30 to R55, R110 to R56, R31 to R57, R111 to R58, R32 to R59, R85 to R6, R112 to R60, R33 to R61, R34 to R62, R113 to R63, R114 to R64, R35 to R65, R115 to R66, R36 to R67, R116 to R68, R37 to R69, R6 to R7, R117 to R70, R38 to R71, R118 to R72, R39 to R73, R119 to R74, R40 to R75, R41 to R76, R120 to R77, R121 to R78, R42 to R79, R86 to R8, R43 to R80, R122 to R81, R123 to R82, R44 to R83, R124 to R84, R7 to R9, RV21 to RV10, RV6 to RV11, RV22 to RV12, RV7 to RV13, RV23 to RV14, RV8 to RV15, RV24 to RV16, RV17 to RV2, RV2 to RV3, RV18 to RV4, RV3 to RV5, RV19 to RV6, RV4 to RV7, RV20 to RV8, RV5 to RV9, U4 to U3, U6 to U4, U8 to U5, U3 to U6, U5 to U7, U7 to U8
Routing:
- net /amp stage/signal out A: track 54.9 -> 79.7 mm
- net GND: track 176.8 -> 163.3 mm
- net Net-(U9B--): track 31.2 -> 29.2 mm
- net Net-(Q4A-B1): track 74.9 -> 73.1 mm
- net +12V: track 482.7 -> 481.9 mm
