File: 15_oct_vca_mixer/15_oct_vca_mixer.kicad_sch (KiCad schematic)
At the start: 13 parts, among them J1 Signal out, U1 TL072

Commit message: fine-tune 15 PCB
Parts:
- added unit 3 of U1
- renumbered C31 to C3, C32 to C4
Connections:
- net +12V: now also U1.8 (V+); no longer U1.8 (V+)
- net -12V: now also U1.4 (V-); no longer U1.4 (V-)
Changed lines of the file:
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@@
 		(in_pos_files yes)
 		(dnp no)
-		(property "Reference" "#PWR0178"
+		(property "Reference" "#PWR06"
 			(at 118.11 173.99 0)
 			(hide yes)
@@
 			(project "15_oct_vca_mixer"
 				(path "/f3e49307-da6e-4072-8a49-1bd21abcb0da"
-					(reference "#PWR0178")
+					(reference "#PWR06")
 					(unit 1)
 				)
@@
 		(dnp no)
 		(fields_autoplaced yes)
-		(property "Reference" "C32"
+		(property "Reference" "C4"
 			(at 105.41 180.3399 0)
 			(show_name no)
@@
 			(project "15_oct_vca_mixer"
 				(path "/f3e49307-da6e-4072-8a49-1bd21abcb0da"
-					(reference "C32")
+					(reference "C4")
 					(unit 1)
 				)
@@
 		(dnp no)
 		(fields_autoplaced yes)
-		(property "Reference" "#PWR05"
+		(property "Reference" "#PWR08"
 			(at 147.32 39.37 0)
 			(hide yes)
@@
 			(project "15_oct_vca_mixer"
 				(path "/f3e49307-da6e-4072-8a49-1bd21abcb0da"
-					(reference "#PWR05")
+					(reference "#PWR08")
 					(unit 1)
 				)
@@
 		(dnp no)
 		(fields_autoplaced yes)
-		(property "Reference" "#PWR06"
+		(property "Reference" "#PWR09"
 			(at 181.61 44.45 0)
 			(hide yes)
@@
 			(project "15_oct_vca_mixer"
 				(path "/f3e49307-da6e-4072-8a49-1bd21abcb0da"
-					(reference "#PWR06")
+					(reference "#PWR09")
 					(unit 1)
 				)
@@
 		(in_pos_files yes)
 		(dnp no)
-		(property "Reference" "#PWR0179"
+		(property "Reference" "#PWR07"
 			(at 118.11 187.96 0)
 			(hide yes)
@@
 			(project "15_oct_vca_mixer"
 				(path "/f3e49307-da6e-4072-8a49-1bd21abcb0da"
-					(reference "#PWR0179")
+					(reference "#PWR07")
 					(unit 1)
 				)
@@
 		(dnp no)
 		(fields_autoplaced yes)
-		(property "Reference" "#PWR0177"
+		(property "Reference" "#PWR04"
 			(at 97.79 184.15 0)
 			(hide yes)
@@
 			(project "15_oct_vca_mixer"
 				(path "/f3e49307-da6e-4072-8a49-1bd21abcb0da"
-					(reference "#PWR0177")
+					(reference "#PWR04")
 					(unit 1)
 				)
@@
 		(dnp no)
 		(fields_autoplaced yes)
-		(property "Reference" "C31"
+		(property "Reference" "C3"
 			(at 105.41 172.7199 0)
 			(show_name no)
@@
 			(project "15_oct_vca_mixer"
 				(path "/f3e49307-da6e-4072-8a49-1bd21abcb0da"
-					(reference "C31")
+					(reference "C3")
 					(unit 1)
 				)
@@
 		(dnp no)
 		(fields_autoplaced yes)
-		(property "Reference" "#PWR04"
+		(property "Reference" "#PWR05"
 			(at 109.22 39.37 0)
 			(hide yes)
@@
 			(project "15_oct_vca_mixer"
 				(path "/f3e49307-da6e-4072-8a49-1bd21abcb0da"
-					(reference "#PWR04")
-					(unit 1)
-				)
+					(reference "#PWR05")
+					(unit 1)
+				)
