File: 15_oct_vca_mixer/apm_stage.kicad_sch (KiCad schematic)
At the start: 68 parts, among them J10 CV in, J11 signal in, J2 CV in, J3 signal in, Q1 BC847BS, Q5 BC847BS, U2 TL072, U4 TL072, U6 TL072, U8 TL072

Commit message: fine-tune 15 PCB
Parts:
- added TP1, TP3: TestPoint, TestPoint:TestPoint_Pad_2.0x2.0mm, symbol Connector:TestPoint
- renumbered C20 to C10, C27 to C11, C28 to C12, C3 to C5, C4 to C6, C5 to C7, C6 to C8, C19 to C9, D7 to D4, J10 to J3, J3 to J4, J11 to J5, Q5 to Q2, R87 to R10, R8 to R11, R88 to R12, R10 to R13, R89 to R14, R11 to R15, R90 to R16, R9 to R17, R91 to R18, R12 to R19, R92 to R20, R13 to R21, R15 to R22, R93 to R23, R94 to R24, R14 to R25, R95 to R26, R16 to R27, R96 to R28, R17 to R29, R97 to R30, R18 to R31, R98 to R32, R19 to R33, R99 to R34, R20 to R35, R21 to R36, R100 to R37, R101 to R38, R22 to R39, R23 to R40, R102 to R41, R103 to R42, R24 to R43, R104 to R44, R85 to R6, R6 to R7, R86 to R8, R7 to R9, RV17 to RV2, RV2 to RV3, RV18 to RV4, RV3 to RV5, RV19 to RV6, RV4 to RV7, RV20 to RV8, U4 to U3, U6 to U4, U8 to U5
Connections:
- net at D3.2 (A), Q1.1 (E1), Q1.4 (E2)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: now also TP3.1
- net at D4.2 (A), Q2.1 (E1), Q2.4 (E2)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: now also TP1.1
