File: 01_as3340_vco/01_as3340_vco.kicad_pcb (KiCad board)
At the start: 2 copper layers, 60 x 108 mm, 100 parts, among them J10 SINE OUT, J3 SYNC IN, J4 FM IN, J5 PWM CV IN, J6 1V per O IN, J7 SQUARE OUT, J8 SAW OUT, J9 TRI OUT, Q1 BC847, Q2 BC847, SW2 SW_SPDT, U1 TL072, U2 AS3340, U3 TL074

Commit message: Normalize resistor footprint, diode and transistor part numbers
Three part choices differed between modules for no reason, which split
them into separate lines in the collective BOM:

- module 03 used the stock Resistor_SMD:R_0805_2012Metric_Pad1.20x1.40mm_
  HandSolder for its 84 resistors, all other modules use the copy in
  lib/kicad/cynthia.pretty ("cynthia:R SMD  0805").  The two footprints
  are geometrically identical (same pads, silk, courtyard and 3D model),
  so the layout of module 03 does not change.
- modules 01 and 02 called their SOD-323 diodes 1N4148; module 03 used
  the correct part number for that package, 1N4148WS.  Now 1N4148WS
  everywhere.  The symbols stay Device:D / Device:D_Small, only the
  value changes.
- modules 02 and 04 used BC848 where 01 uses BC847.  Both are NPN SOT-23
  with identical symbols and the same datasheet; switched to BC847,
  including the cached lib_symbols entry and the description (45V Vce).

Schematics, boards and netlists are updated consistently.

Collective BOM after the change: 1N4148WS 12x (was 8x 1N4148 + 4x
1N4148WS), BC847 4x (was 2x BC847 + 2x BC848), and all 152 resistors on
one footprint.

Co-Authored-By: Claude Opus 5 <noreply@anthropic.com>
Claude-Session: https://claude.ai/code/session_01RDRvK2YhNsxKhLToRaEtAA
Parts:
- D1, D2: value 1N4148 -> 1N4148WS
Changed lines of the file:
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@@
 			)
 		)
-		(property "Value" "1N4148"
+		(property "Value" "1N4148WS"
 			(at 0.1 1.9 90)
 			(layer "F.Fab")
@@
 			)
 		)
-		(property "Value" "1N4148"
+		(property "Value" "1N4148WS"
 			(at 0.1 1.9 90)
 			(layer "F.Fab")
