File: 01_as3340_vco/01_as3340_vco.kicad_sch (KiCad schematic)
At the start: 100 parts, among them J10 SINE OUT, J3 SYNC IN, J4 FM IN, J5 PWM CV IN, J6 1V per O IN, J7 SQUARE OUT, J8 SAW OUT, J9 TRI OUT, Q1 BC847, Q2 BC847, SW2 SW_SPDT, U1 TL072, U2 AS3340, U3 TL074

Commit message: Normalize resistor footprint, diode and transistor part numbers
Three part choices differed between modules for no reason, which split
them into separate lines in the collective BOM:

- module 03 used the stock Resistor_SMD:R_0805_2012Metric_Pad1.20x1.40mm_
  HandSolder for its 84 resistors, all other modules use the copy in
  lib/kicad/cynthia.pretty ("cynthia:R SMD  0805").  The two footprints
  are geometrically identical (same pads, silk, courtyard and 3D model),
  so the layout of module 03 does not change.
- modules 01 and 02 called their SOD-323 diodes 1N4148; module 03 used
  the correct part number for that package, 1N4148WS.  Now 1N4148WS
  everywhere.  The symbols stay Device:D / Device:D_Small, only the
  value changes.
- modules 02 and 04 used BC848 where 01 uses BC847.  Both are NPN SOT-23
  with identical symbols and the same datasheet; switched to BC847,
  including the cached lib_symbols entry and the description (45V Vce).

Schematics, boards and netlists are updated consistently.

Collective BOM after the change: 1N4148WS 12x (was 8x 1N4148 + 4x
1N4148WS), BC847 4x (was 2x BC847 + 2x BC848), and all 152 resistors on
one footprint.

Co-Authored-By: Claude Opus 5 <noreply@anthropic.com>
Claude-Session: https://claude.ai/code/session_01RDRvK2YhNsxKhLToRaEtAA
Parts:
- D1, D2: value 1N4148 -> 1N4148WS
Changed lines of the file:
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@@
 			)
 		)
-		(property "Value" "1N4148"
+		(property "Value" "1N4148WS"
 			(at 95.25 71.1199 90)
 			(show_name no)
@@
 			)
 		)
-		(property "Value" "1N4148"
+		(property "Value" "1N4148WS"
 			(at 95.25 78.7399 90)
 			(show_name no)

Commit message: Add a true hard-reset input to the AS3340 VCO
The AS3340's hard sync input (pin 6) feeds the internal charge/discharge
state comparator through a 6.3k resistor; it has no path to pin 11 (CAP).
Hard sync therefore reverses the ramp direction from wherever it happens
to be rather than resetting the timing capacitor, which the "Output
Waveforms" figure on page 3 of the datasheet shows directly: the triangle
turns around mid-slope and the sawtooth gets a mid-ramp notch. That is a
usable sync flavour but no good as an LFO restart.

Add a RESET IN jack that pulls the timing cap to 0 V, so triangle, saw and
square all restart from a defined phase in both range-switch positions:

  J11 -> D6 -> 100k pulldown -> U1C comparator (2.09 V threshold from the
  same 100k/22k divider used in module 02, hysteresis via R56) -> R52/C10
  differentiator -> Q3 base -> Q3 shorts the CAP node through R51 100R.

Because the comparator supplies a fixed-amplitude edge, the ~15 us
discharge pulse no longer depends on the trigger's amplitude or slew. The
timing caps are small (820 pF audio, 10 nF LFO), so one fixed pulse covers
both ranges. D5 clamps Q3's base against the comparator's negative swing.

Every op-amp section was already in use, so U1 becomes a TL074 (SOIC-14):
U1A and U1B keep their pin numbers, only the power pins move (V+ 8 -> 4,
V- 4 -> 11). U1C is the comparator, U1D is tied off as a grounded
follower. The module now uses two TL074s and no TL072.

The A4 sheet had no free area left that could hold the new block without
overlapping the title block, so the schematic is now A3.

The netlist and PCB still need regenerating from KiCad; see the README.

Co-Authored-By: Claude Opus 5 <noreply@anthropic.com>
Claude-Session: https://claude.ai/code/session_01Sn5onQfMWSZqYkeJqqv5h8
Parts:
- added C10: 330pF, cynthia:C SMD 0805, symbol Device:C_Small
- added D5, D6: 1N4148WS, Diode_SMD:D_SOD-323_HandSoldering, symbol Device:D_Small
- added J11: RESET IN, cynthia:3.5mm jack mono switched, symbol Connector_Audio:AudioJack2_SwitchT
- added Q3: BC847, Package_TO_SOT_SMD:SOT-23, symbol Transistor_BJT:BC847
- added R51: 100R, cynthia:R SMD 0805, symbol Device:R_Small
- added R52: 10k, cynthia:R SMD 0805, symbol Device:R_Small
- added R53, R54, R55, R57: 100k, cynthia:R SMD 0805, symbol Device:R_Small
- added R56: 2M2, cynthia:R SMD 0805, symbol Device:R_Small
- added R58: 22k, cynthia:R SMD 0805, symbol Device:R_Small
- added unit 4 of U1
- added unit 3 of U1
- U1: value TL072 -> TL074; footprint cynthia:SOIC-8_3.9x4.9mm_P1.27mm -> cynthia:SOIC-14_3.9x8.7mm_P1.27mm; symbol Amplifier_Operational:TL072 -> Amplifier_Operational:TL074
Connections:
- net +12V: now also U1.4 (V+), R57.1; no longer U1.8 (V+)
- net -12V: now also U1.11 (V-); no longer U1.4 (V-)
- net GND: now also D5.2 (A), J11.S, J11.TN, Q3.2 (E), R53.2, R54.2, R58.2, U1.12 (+)
- net CAP: now reaches SW2.2 (B), U2.11 (CAP)
- net CAP: now also R51.1
- new net: C10.2, D5.1 (K), Q3.1 (B), R53.1
- new net: Q3.3 (C), R51.2
- new net: D6.2 (A), J11.T
- new net: R52.1, R56.2, U1.8
- new net: C10.1, R52.2
- new net: D6.1 (K), R54.1, R55.1
- new net: R55.2, R56.1, U1.10 (+)
- new net: R57.2, R58.1, U1.9 (-)
- new net: U1.13 (-), U1.14
