File: 03_quad_vca_mixer/03_quad_vca_mixer.kicad_pcb (KiCad board)
At the start: 2 copper layers, 70 x 100 mm, 153 parts, among them J1 Signal out, J2 CV in, J3 CV in, J4 signal in, J5 signal in, J6 CV in, J7 CV in, J8 signal in, J9 signal in, Q1 BC847BS, Q2 BC847BS, Q3 BC847BS, Q4 BC847BS, U1 TL072, U2 TL072, U3 TL072, U4 TL072, U5 TL072, U6 TL072, U7 TL072, U8 TL072, U9 TL072

Commit message: Normalize resistor footprint, diode and transistor part numbers
Three part choices differed between modules for no reason, which split
them into separate lines in the collective BOM:

- module 03 used the stock Resistor_SMD:R_0805_2012Metric_Pad1.20x1.40mm_
  HandSolder for its 84 resistors, all other modules use the copy in
  lib/kicad/cynthia.pretty ("cynthia:R SMD  0805").  The two footprints
  are geometrically identical (same pads, silk, courtyard and 3D model),
  so the layout of module 03 does not change.
- modules 01 and 02 called their SOD-323 diodes 1N4148; module 03 used
  the correct part number for that package, 1N4148WS.  Now 1N4148WS
  everywhere.  The symbols stay Device:D / Device:D_Small, only the
  value changes.
- modules 02 and 04 used BC848 where 01 uses BC847.  Both are NPN SOT-23
  with identical symbols and the same datasheet; switched to BC847,
  including the cached lib_symbols entry and the description (45V Vce).

Schematics, boards and netlists are updated consistently.

Collective BOM after the change: 1N4148WS 12x (was 8x 1N4148 + 4x
1N4148WS), BC847 4x (was 2x BC847 + 2x BC848), and all 152 resistors on
one footprint.

Co-Authored-By: Claude Opus 5 <noreply@anthropic.com>
Claude-Session: https://claude.ai/code/session_01RDRvK2YhNsxKhLToRaEtAA
Parts:
- R1, R10, R11, R12, R13, R14, R15, R16, R17, R18, R19, R2, R20, R21, R22, R23, R24, R25, R26, R27, R28, R29, R3, R30, R31, R32, R33, R34, R35, R36, R37, R38, R39, R4, R40, R41, R42, R43, R44, R45, R46, R47, R48, R49, R5, R50, R51, R52, R53, R54, R55, R56, R57, R58, R59, R6, R60, R61, R62, R63, R64, R65, R66, R67, R68, R69, R7, R70, R71, R72, R73, R74, R75, R76, R77, R78, R79, R8, R80, R81, R82, R83, R84, R9: footprint Resistor_SMD:R_0805_2012Metric_Pad1.20x1.40mm_HandSolder -> cynthia:R SMD 0805
