File: 03_quad_vca_mixer/03_quad_vca_mixer.kicad_sch (KiCad schematic)
At the start: 13 parts, among them J1 Signal out, U1 TL072

Commit message: Normalize resistor footprint, diode and transistor part numbers
Three part choices differed between modules for no reason, which split
them into separate lines in the collective BOM:

- module 03 used the stock Resistor_SMD:R_0805_2012Metric_Pad1.20x1.40mm_
  HandSolder for its 84 resistors, all other modules use the copy in
  lib/kicad/cynthia.pretty ("cynthia:R SMD  0805").  The two footprints
  are geometrically identical (same pads, silk, courtyard and 3D model),
  so the layout of module 03 does not change.
- modules 01 and 02 called their SOD-323 diodes 1N4148; module 03 used
  the correct part number for that package, 1N4148WS.  Now 1N4148WS
  everywhere.  The symbols stay Device:D / Device:D_Small, only the
  value changes.
- modules 02 and 04 used BC848 where 01 uses BC847.  Both are NPN SOT-23
  with identical symbols and the same datasheet; switched to BC847,
  including the cached lib_symbols entry and the description (45V Vce).

Schematics, boards and netlists are updated consistently.

Collective BOM after the change: 1N4148WS 12x (was 8x 1N4148 + 4x
1N4148WS), BC847 4x (was 2x BC847 + 2x BC848), and all 152 resistors on
one footprint.

Co-Authored-By: Claude Opus 5 <noreply@anthropic.com>
Claude-Session: https://claude.ai/code/session_01RDRvK2YhNsxKhLToRaEtAA
Parts:
- R1, R2, R3, R4: footprint Resistor_SMD:R_0805_2012Metric_Pad1.20x1.40mm_HandSolder -> cynthia:R SMD 0805
Changed lines of the file:
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@@
 			)
 		)
-		(property "Footprint" "Resistor_SMD:R_0805_2012Metric_Pad1.20x1.40mm_HandSolder"
+		(property "Footprint" "cynthia:R SMD  0805"
 			(at 133.35 37.338 90)
 			(hide yes)
@@
 			)
 		)
-		(property "Footprint" "Resistor_SMD:R_0805_2012Metric_Pad1.20x1.40mm_HandSolder"
+		(property "Footprint" "cynthia:R SMD  0805"
 			(at 172.72 37.338 90)
 			(hide yes)
@@
 			)
 		)
-		(property "Footprint" "Resistor_SMD:R_0805_2012Metric_Pad1.20x1.40mm_HandSolder"
+		(property "Footprint" "cynthia:R SMD  0805"
 			(at 116.84 47.498 90)
 			(hide yes)
@@
 			)
 		)
-		(property "Footprint" "Resistor_SMD:R_0805_2012Metric_Pad1.20x1.40mm_HandSolder"
+		(property "Footprint" "cynthia:R SMD  0805"
 			(at 154.94 47.498 90)
 			(hide yes)
