File: 04_diode_ladder_vcf/04_diode_ladder_vcf.kicad_pcb (KiCad board)
At the start: 2 copper layers, 30 x 100 mm, 66 parts, among them J1 Audio In, J2 Cutoff CV In, J3 Audio Out, Q1 BC848, Q2 BC848, U1 TL074

Commit message: Normalize resistor footprint, diode and transistor part numbers
Three part choices differed between modules for no reason, which split
them into separate lines in the collective BOM:

- module 03 used the stock Resistor_SMD:R_0805_2012Metric_Pad1.20x1.40mm_
  HandSolder for its 84 resistors, all other modules use the copy in
  lib/kicad/cynthia.pretty ("cynthia:R SMD  0805").  The two footprints
  are geometrically identical (same pads, silk, courtyard and 3D model),
  so the layout of module 03 does not change.
- modules 01 and 02 called their SOD-323 diodes 1N4148; module 03 used
  the correct part number for that package, 1N4148WS.  Now 1N4148WS
  everywhere.  The symbols stay Device:D / Device:D_Small, only the
  value changes.
- modules 02 and 04 used BC848 where 01 uses BC847.  Both are NPN SOT-23
  with identical symbols and the same datasheet; switched to BC847,
  including the cached lib_symbols entry and the description (45V Vce).

Schematics, boards and netlists are updated consistently.

Collective BOM after the change: 1N4148WS 12x (was 8x 1N4148 + 4x
1N4148WS), BC847 4x (was 2x BC847 + 2x BC848), and all 152 resistors on
one footprint.

Co-Authored-By: Claude Opus 5 <noreply@anthropic.com>
Claude-Session: https://claude.ai/code/session_01RDRvK2YhNsxKhLToRaEtAA
Parts:
- Q1, Q2: value BC848 -> BC847
Changed lines of the file:
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@@
 			)
 		)
-		(property "Value" "BC848"
+		(property "Value" "BC847"
 			(at 0 2.4 0)
 			(layer "F.Fab")
@@
 			)
 		)
-		(property "Description" "0.1A Ic, 30V Vce, NPN Transistor, SOT-23"
+		(property "Description" "0.1A Ic, 45V Vce, NPN Transistor, SOT-23"
 			(at 0 0 0)
 			(layer "F.Fab")
@@
 			)
 		)
-		(property "Value" "BC848"
+		(property "Value" "BC847"
 			(at 0 2.4 0)
 			(layer "F.Fab")
@@
 			)
 		)
-		(property "Description" "0.1A Ic, 30V Vce, NPN Transistor, SOT-23"
+		(property "Description" "0.1A Ic, 45V Vce, NPN Transistor, SOT-23"
 			(at 0 0 0)
 			(layer "F.Fab")
