File: 04_diode_ladder_vcf/04_diode_ladder_vcf.kicad_sch (KiCad schematic)
At the start: 66 parts, among them J1 Audio In, J2 Cutoff CV In, J3 Audio Out, Q1 BC848, Q2 BC848, U1 TL074

Commit message: Normalize resistor footprint, diode and transistor part numbers
Three part choices differed between modules for no reason, which split
them into separate lines in the collective BOM:

- module 03 used the stock Resistor_SMD:R_0805_2012Metric_Pad1.20x1.40mm_
  HandSolder for its 84 resistors, all other modules use the copy in
  lib/kicad/cynthia.pretty ("cynthia:R SMD  0805").  The two footprints
  are geometrically identical (same pads, silk, courtyard and 3D model),
  so the layout of module 03 does not change.
- modules 01 and 02 called their SOD-323 diodes 1N4148; module 03 used
  the correct part number for that package, 1N4148WS.  Now 1N4148WS
  everywhere.  The symbols stay Device:D / Device:D_Small, only the
  value changes.
- modules 02 and 04 used BC848 where 01 uses BC847.  Both are NPN SOT-23
  with identical symbols and the same datasheet; switched to BC847,
  including the cached lib_symbols entry and the description (45V Vce).

Schematics, boards and netlists are updated consistently.

Collective BOM after the change: 1N4148WS 12x (was 8x 1N4148 + 4x
1N4148WS), BC847 4x (was 2x BC847 + 2x BC848), and all 152 resistors on
one footprint.

Co-Authored-By: Claude Opus 5 <noreply@anthropic.com>
Claude-Session: https://claude.ai/code/session_01RDRvK2YhNsxKhLToRaEtAA
Parts:
- Q1, Q2: value BC848 -> BC847; symbol Transistor_BJT:BC848 -> Transistor_BJT:BC847
Changed lines of the file:
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@@
 	)
 	(symbol
-		(lib_id "Transistor_BJT:BC848")
+		(lib_id "Transistor_BJT:BC847")
 		(at 156.21 133.35 0)
 		(mirror y)
@@
 			)
 		)
-		(property "Value" "BC848"
+		(property "Value" "BC847"
 			(at 151.13 134.6199 0)
 			(show_name no)
@@
 			)
 		)
-		(property "Description" "0.1A Ic, 30V Vce, NPN Transistor, SOT-23"
+		(property "Description" "0.1A Ic, 45V Vce, NPN Transistor, SOT-23"
 			(at 156.21 133.35 0)
 			(hide yes)
@@
 	)
 	(symbol
-		(lib_id "Transistor_BJT:BC848")
+		(lib_id "Transistor_BJT:BC847")
 		(at 121.92 133.35 0)
 		(unit 1)
@@
 			)
 		)
-		(property "Value" "BC848"
+		(property "Value" "BC847"
 			(at 127 134.6199 0)
 			(show_name no)
@@
 			)
 		)
-		(property "Description" "0.1A Ic, 30V Vce, NPN Transistor, SOT-23"
+		(property "Description" "0.1A Ic, 45V Vce, NPN Transistor, SOT-23"
 			(at 121.92 133.35 0)
 			(hide yes)

Commit message: Use BC857 as the PNP complement and give module 04 real diodes
Follow-up to the part normalization:

- module 02 Q1/Q3 were BC858, the complement of the BC848 they were
  paired with.  Now that the NPNs are BC847, their complement is BC857
  (45V instead of 30V Vce), so only one NPN/PNP pair needs stocking.
  Same symbol, same onsemi BC856..BC860 datasheet; the cached
  lib_symbols entry and the description were updated too.
- module 04's ladder diodes D1-D10 had no part number at all (value "D")
  and sat on cynthia:D SMD 0805, while every other module uses 1N4148WS
  in SOD-323.  They are now 1N4148WS on Diode_SMD:D_SOD-323_HandSoldering.

The module 04 board is not updated: unlike the 0805 resistor swap, these
two footprints have different pad geometry, so the footprints have to be
replaced by KiCad itself via Update PCB from Schematic.  The board has no
routing yet, so nothing is lost.

Co-Authored-By: Claude Opus 5 <noreply@anthropic.com>
Claude-Session: https://claude.ai/code/session_01RDRvK2YhNsxKhLToRaEtAA
Parts:
- D1, D10, D2, D3, D4, D5, D6, D7, D8, D9: value D -> 1N4148WS; footprint cynthia:D SMD 0805 -> Diode_SMD:D_SOD-323_HandSoldering
Changed lines of the file:
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@@
 			)
 		)
-		(property "Value" "D"
+		(property "Value" "1N4148WS"
 			(at 172.72 86.36 0)
 			(show_name no)
@@
 			)
 		)
-		(property "Footprint" "cynthia:D SMD 0805"
+		(property "Footprint" "Diode_SMD:D_SOD-323_HandSoldering"
 			(at 172.72 90.17 0)
 			(hide yes)
@@
 			)
 		)
-		(property "Value" "D"
+		(property "Value" "1N4148WS"
 			(at 134.62 86.36 0)
 			(show_name no)
@@
 			)
 		)
-		(property "Footprint" "cynthia:D SMD 0805"
+		(property "Footprint" "Diode_SMD:D_SOD-323_HandSoldering"
 			(at 134.62 90.17 0)
 			(hide yes)
@@
 			)
 		)
-		(property "Value" "D"
+		(property "Value" "1N4148WS"
 			(at 149.86 86.36 0)
 			(show_name no)
@@
 			)
 		)
-		(property "Footprint" "cynthia:D SMD 0805"
+		(property "Footprint" "Diode_SMD:D_SOD-323_HandSoldering"
 			(at 149.86 90.17 0)
 			(hide yes)
@@
 			)
 		)
-		(property "Value" "D"
+		(property "Value" "1N4148WS"
 			(at 119.38 86.36 0)
 			(show_name no)
@@
 			)
 		)
-		(property "Footprint" "cynthia:D SMD 0805"
+		(property "Footprint" "Diode_SMD:D_SOD-323_HandSoldering"
 			(at 119.38 90.17 0)
 			(hide yes)
@@
 			)
 		)
-		(property "Value" "D"
+		(property "Value" "1N4148WS"
 			(at 127 86.36 0)
 			(show_name no)
@@
 			)
 		)
-		(property "Footprint" "cynthia:D SMD 0805"
+		(property "Footprint" "Diode_SMD:D_SOD-323_HandSoldering"
 			(at 127 90.17 0)
 			(hide yes)
@@
 			)
 		)
-		(property "Value" "D"
+		(property "Value" "1N4148WS"
 			(at 142.24 86.36 0)
 			(show_name no)
@@
 			)
 		)
-		(property "Footprint" "cynthia:D SMD 0805"
+		(property "Footprint" "Diode_SMD:D_SOD-323_HandSoldering"
 			(at 142.24 90.17 0)
 			(hide yes)
@@
 			)
 		)
-		(property "Value" "D"
+		(property "Value" "1N4148WS"
 			(at 104.14 86.36 0)
 			(show_name no)
@@
 			)
 		)
-		(property "Footprint" "cynthia:D SMD 0805"
+		(property "Footprint" "Diode_SMD:D_SOD-323_HandSoldering"
 			(at 104.14 90.17 0)
 			(hide yes)
@@
 			)
 		)
-		(property "Value" "D"
+		(property "Value" "1N4148WS"
 			(at 165.1 86.36 0)
 			(show_name no)
@@
 			)
 		)
-		(property "Footprint" "cynthia:D SMD 0805"
+		(property "Footprint" "Diode_SMD:D_SOD-323_HandSoldering"
 			(at 165.1 90.17 0)
 			(hide yes)
@@
 			)
 		)
-		(property "Value" "D"
+		(property "Value" "1N4148WS"
 			(at 157.48 86.36 0)
 			(show_name no)
@@
 			)
 		)
-		(property "Footprint" "cynthia:D SMD 0805"
+		(property "Footprint" "Diode_SMD:D_SOD-323_HandSoldering"
 			(at 157.48 90.17 0)
 			(hide yes)
@@
 			)
 		)
-		(property "Value" "D"
+		(property "Value" "1N4148WS"
 			(at 111.76 86.36 0)
 			(show_name no)
@@
 			)
 		)
-		(property "Footprint" "cynthia:D SMD 0805"
+		(property "Footprint" "Diode_SMD:D_SOD-323_HandSoldering"
 			(at 111.76 90.17 0)
 			(hide yes)
