File: 02_loop_env/02_loop_env.kicad_pcb (KiCad board)
At the start: 2 copper layers, 30 x 100 mm, 55 parts, among them J1 gate in 1, J2 End of Cycle Out, J3 env out 1, Q1 BC858, Q2 BC848, Q3 BC858, Q4 BC848, SW1 Manual Gate, SW2 Gate/Loop, SW4 Normal/Inverted, U1 TL074, U2 TL072

Commit message: Normalize resistor footprint, diode and transistor part numbers
Three part choices differed between modules for no reason, which split
them into separate lines in the collective BOM:

- module 03 used the stock Resistor_SMD:R_0805_2012Metric_Pad1.20x1.40mm_
  HandSolder for its 84 resistors, all other modules use the copy in
  lib/kicad/cynthia.pretty ("cynthia:R SMD  0805").  The two footprints
  are geometrically identical (same pads, silk, courtyard and 3D model),
  so the layout of module 03 does not change.
- modules 01 and 02 called their SOD-323 diodes 1N4148; module 03 used
  the correct part number for that package, 1N4148WS.  Now 1N4148WS
  everywhere.  The symbols stay Device:D / Device:D_Small, only the
  value changes.
- modules 02 and 04 used BC848 where 01 uses BC847.  Both are NPN SOT-23
  with identical symbols and the same datasheet; switched to BC847,
  including the cached lib_symbols entry and the description (45V Vce).

Schematics, boards and netlists are updated consistently.

Collective BOM after the change: 1N4148WS 12x (was 8x 1N4148 + 4x
1N4148WS), BC847 4x (was 2x BC847 + 2x BC848), and all 152 resistors on
one footprint.

Co-Authored-By: Claude Opus 5 <noreply@anthropic.com>
Claude-Session: https://claude.ai/code/session_01RDRvK2YhNsxKhLToRaEtAA
Parts:
- D1, D4, D5, D6, D7, D8: value 1N4148 -> 1N4148WS
- Q2, Q4: value BC848 -> BC847
Changed lines of the file:
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@@
 			)
 		)
-		(property "Value" "1N4148"
+		(property "Value" "1N4148WS"
 			(at 0.1 -1.9 270)
 			(layer "B.Fab")
@@
 			)
 		)
-		(property "Value" "BC848"
+		(property "Value" "BC847"
 			(at 0 -2.4 0)
 			(layer "B.Fab")
@@
 			)
 		)
-		(property "Description" "0.1A Ic, 30V Vce, NPN Transistor, SOT-23"
+		(property "Description" "0.1A Ic, 45V Vce, NPN Transistor, SOT-23"
 			(at 0 0 0)
 			(layer "B.Fab")
@@
 			)
 		)
-		(property "Value" "BC848"
+		(property "Value" "BC847"
 			(at 0 -2.4 0)
 			(layer "B.Fab")
@@
 			)
 		)
-		(property "Description" "0.1A Ic, 30V Vce, NPN Transistor, SOT-23"
+		(property "Description" "0.1A Ic, 45V Vce, NPN Transistor, SOT-23"
 			(at 0 0 0)
 			(layer "B.Fab")
@@
 			)
 		)
-		(property "Value" "1N4148"
+		(property "Value" "1N4148WS"
 			(at 0.1 -1.9 90)
 			(layer "B.Fab")
@@
 			)
 		)
-		(property "Value" "1N4148"
+		(property "Value" "1N4148WS"
 			(at 0.1 -1.9 0)
 			(layer "B.Fab")
@@
 			)
 		)
-		(property "Value" "1N4148"
+		(property "Value" "1N4148WS"
 			(at 0.1 -1.9 0)
 			(layer "B.Fab")
@@
 			)
 		)
-		(property "Value" "1N4148"
+		(property "Value" "1N4148WS"
 			(at 0.1 -1.9 0)
 			(layer "B.Fab")
@@
 			)
 		)
-		(property "Value" "1N4148"
+		(property "Value" "1N4148WS"
 			(at 0.1 -1.9 90)
 			(layer "B.Fab")

Commit message: Use BC857 as the PNP complement and give module 04 real diodes
Follow-up to the part normalization:

- module 02 Q1/Q3 were BC858, the complement of the BC848 they were
  paired with.  Now that the NPNs are BC847, their complement is BC857
  (45V instead of 30V Vce), so only one NPN/PNP pair needs stocking.
  Same symbol, same onsemi BC856..BC860 datasheet; the cached
  lib_symbols entry and the description were updated too.
- module 04's ladder diodes D1-D10 had no part number at all (value "D")
  and sat on cynthia:D SMD 0805, while every other module uses 1N4148WS
  in SOD-323.  They are now 1N4148WS on Diode_SMD:D_SOD-323_HandSoldering.

The module 04 board is not updated: unlike the 0805 resistor swap, these
two footprints have different pad geometry, so the footprints have to be
replaced by KiCad itself via Update PCB from Schematic.  The board has no
routing yet, so nothing is lost.

Co-Authored-By: Claude Opus 5 <noreply@anthropic.com>
Claude-Session: https://claude.ai/code/session_01RDRvK2YhNsxKhLToRaEtAA
Parts:
- Q1, Q3: value BC858 -> BC857
Changed lines of the file:
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@@
 			)
 		)
-		(property "Value" "BC858"
+		(property "Value" "BC857"
 			(at 0 -2.4 0)
 			(layer "B.Fab")
@@
 			)
 		)
-		(property "Description" "0.1A Ic, 30V Vce, PNP Transistor, SOT-23"
+		(property "Description" "0.1A Ic, 45V Vce, PNP Transistor, SOT-23"
 			(at 0 0 0)
 			(layer "B.Fab")
@@
 			)
 		)
-		(property "Value" "BC858"
+		(property "Value" "BC857"
 			(at 0 -2.4 0)
 			(layer "B.Fab")
@@
 			)
 		)
-		(property "Description" "0.1A Ic, 30V Vce, PNP Transistor, SOT-23"
+		(property "Description" "0.1A Ic, 45V Vce, PNP Transistor, SOT-23"
 			(at 0 0 0)
 			(layer "B.Fab")
