File: 02_loop_env/02_loop_env.kicad_sch (KiCad schematic)
At the start: 55 parts, among them J1 gate in 1, J2 End of Cycle Out, J3 env out 1, Q1 BC857, Q2 BC847, Q3 BC857, Q4 BC847, SW1 Manual Gate, SW2 Gate/Loop, SW4 Normal/Inverted, U1 TL074, U2 TL072

Commit message: updated 02
Parts:
- removed D6: 1N4148WS, Diode_SMD:D_SOD-323_HandSoldering, symbol Device:D
- added R_E2: 3.3k, cynthia:R SMD 0805, symbol Device:R
- R13: value 33k -> 150k
Connections:
- net -12V: now also RV2.1
- net at R4.2, TP1.1, U1.10 (+)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: no longer SW2.1 (A)
- net at RV2.2, RV2.3, SW3.5: now also R_E2.2
- net at Q2.2 (E): now also R_E2.1
- net at R10.2, RV1.1: no longer RV2.1
- new net: R15.1, SW4.1 (A)
- new net: U2.1, U2.2 (-)
- now unconnected: U1.13 (-)
- no-connect marks 4 -> 7
Other:
- moved on the sheet: R15, R16, U2B

Commit message: design for 02 with LM13700
Parts:
- removed C7, C8: 100nF, cynthia:C SMD 0805, symbol Device:C
- removed C9: 1uF, Capacitor_THT:C_Rect_L7.0mm_W6.5mm_P5.00mm, symbol Device:C
- removed J1: gate in 1, cynthia:3.5mm jack mono switched, symbol Connector_Audio:AudioJack2_SwitchT
- removed J2: End of Cycle Out, cynthia:3.5mm jack mono switched, symbol Connector_Audio:AudioJack2_SwitchT
- removed J3: env out 1, cynthia:3.5mm jack mono switched, symbol Connector_Audio:AudioJack2_SwitchT
- removed Q1, Q3: BC857, Package_TO_SOT_SMD:SOT-23, symbol Transistor_BJT:BC857
- removed Q2, Q4: BC847, Package_TO_SOT_SMD:SOT-23, symbol Transistor_BJT:BC847
- removed R_E2: 3.3k, cynthia:R SMD 0805, symbol Device:R
- removed SW2: Gate/Loop, cynthia:switch_spdt, symbol Switch:SW_SPDT
- removed SW3: (no value), cynthia:switch_dpdt, symbol cynthia:SW_DPDT
- removed SW4: Normal/Inverted, cynthia:switch_spdt, symbol Switch:SW_SPDT
- removed TP1, TP2: TestPoint, TestPoint:TestPoint_Pad_2.0x2.0mm, symbol Connector:TestPoint
- removed U1: TL074, cynthia:SOIC-14_3.9x8.7mm_P1.27mm, symbol Amplifier_Operational:TL074
- removed U2: TL072, cynthia:SOIC-8_3.9x4.9mm_P1.27mm, symbol Amplifier_Operational:TL072
- added C10, C7, C8, C9: 100nF, cynthia:C SMD 0805, symbol Device:C_Small
- added C11: 100nF, Capacitor_THT:C_Rect_L11.5mm_W5.0mm_P10.00mm_MKT, symbol Device:C_Small
- added D2: 1N4148WS, Diode_SMD:D_SOD-323_HandSoldering, symbol Device:D
- added J1, J2, J3, J4, J6: (no value), cynthia:3.5mm thonk jack socket mono switched, symbol cynthia:3.5mm jack mono switched
- added Q1, Q5: BC847, Package_TO_SOT_SMD:SOT-23, symbol Transistor_BJT:BC847
- added Q2, Q3: BCM857BS, Package_TO_SOT_SMD:SOT-363_SC-70-6, symbol Transistor_BJT:BC857BS
- added Q4: BC857, Package_TO_SOT_SMD:SOT-23, symbol Transistor_BJT:BC857
- added R19: 56k, cynthia:R SMD 0805, symbol Device:R
- added R20: 18k, cynthia:R SMD 0805, symbol Device:R
- added R21: 220R, cynthia:R SMD 0805, symbol Device:R
- added R22, R31: 10k, cynthia:R SMD 0805, symbol Device:R
- added R23, R24, R25, R26, R33, R36: 100k, cynthia:R SMD 0805, symbol Device:R
- added R27, R28: 1.5m, cynthia:R SMD 0805, symbol Device:R
- added R29, R30: 82k, cynthia:R SMD 0805, symbol Device:R
- added R34, R35: 15k, cynthia:R SMD 0805, symbol Device:R
- added R37, R38: 510R, cynthia:R SMD 0805, symbol Device:R
- added R39, R40: 1k, cynthia:R SMD 0805, symbol Device:R
- added R41, R42: 7.5k, cynthia:R SMD 0805, symbol Device:R
- added RV3, RV4: 10k, cynthia:potientiometer, symbol Device:R_Potentiometer
- added SW2: SW_DPDT_x2, symbol Switch:SW_DPDT_x2
- added SW3: Normal/Inverted, cynthia:switch_spdt, symbol Switch:SW_SPDT
- added U1, U3: TL072, cynthia:SOIC-8_3.9x4.9mm_P1.27mm, symbol Amplifier_Operational:TL072
- added U4: TL074, cynthia:SOIC-14_3.9x8.7mm_P1.27mm, symbol Amplifier_Operational:TL074
- added U5: LM13700, cynthia:SOIC-16_3.9x9.9mm_P1.27mm, symbol Amplifier_Operational:LM13700
- D8: value 1N4148WS -> BAS416
- R10: value 1k -> 150k
- R11: value 10k -> 100k
- R13: value 150k -> 1k
- R14: value 8.2k -> 4.7k
- R16: value 100k -> 39k
- R17, R9: value 1k -> 10k
- R18: value 1k -> 4.7k
- R4: value 100k -> 9.1k
- R5: value 100k -> 2.2m
- R6: value 100k -> 160k
- R7: value 22k -> 47k
- R8: value 100k -> 10k
- RV1: value 1M -> 5k
- RV2: value 1M -> 10k
- renumbered D2 to D3, D3 to D4, D4 to D6
Connections:
- net +12V: now also R14.2, R3.2, C7.2, C9.2, Q5.3 (C), R19.2, R27.2, R28.2, R41.2, R42.2, U1.8 (V+), U3.8 (V+), U4.4 (V+), U5.11 (V+); no longer R1.2, R11.2, R13.2
- net -12V: now also RV2.3, C10.1, C8.1, Q4.3 (C), RV3.3, U1.4 (V-), U3.4 (V-), U4.11 (V-), U5.6 (V-); no longer RV2.1
- net GND: now also R1.1, R15.1, R4.1, RV2.1, C10.2, C11.1, C7.1, C8.2, C9.1, J1.S, J1.TN, J2.S, J3.S, J3.TN, J4.S, J4.TN, J6.S, Q1.2 (E), Q2.3 (C2), Q2.5 (B2), Q3.3 (C2), Q3.5 (B2), R20.1, R31.1, R37.1, R38.1, RV3.1, U3.3 (+), U3.5 (+), U4.12 (+), U4.3 (+); no longer R14.1, R2.1, R3.1, R8.1
- net at R11.1, R12.2: now also Q1.1 (B)
- net at R18.1: now also D7.1 (K)
- net BASE_RELEASE: now reaches R17.2
- net BASE_RELEASE: now also Q3.2 (B1), R35.2, R38.2
- net at R16.2: now also RV1.1, R19.1, R20.2, U5.14 (+)
- net at D8.2 (A): now also U4.1; no longer D7.1 (K)
- net at D6.2 (A): now also R11.2, R16.1, SW2.2 (B)
- net at R4.2: now also R3.1, U1.2 (-)
- net at R9.1: now also R22.1, U4.10 (+), U4.6 (-), U4.7
- net at R15.2: now also R13.2, J2.T; no longer R16.1
- net at R13.1: now also D5.1 (K); no longer R14.2
- net at RV2.2: now also R23.1; no longer RV2.3
- net at D7.2 (A): now also R14.1, Q1.3 (C)
- net BASE_ATTACK: now reaches R18.2
- net BASE_ATTACK: now also Q2.2 (B1), R34.2, R37.2
- net at R9.2: now also R8.2, U1.6 (-)
- net at R6.1, R7.2: now also R10.1, U1.5 (+)
- net at D1.1 (K), SW1.1: now also R1.2, R2.1; no longer R3.2, R5.1
- net at R5.2: now also SW2.3 (C), SW2.6 (C), U1.1
- net at R10.2: now also D5.2 (A), SW2.1 (A), U1.7; no longer RV1.1
- net at D1.2 (A): now also J1.T
- net at D6.1 (K): now also R17.1; no longer R8.2
- net at RV1.2, RV1.3: now also R21.2; no longer D5.2 (A)
- net at D8.1 (K): now also C11.2, U4.2 (-), U4.5 (+), U5.12
- net at D10.2 (A), D9.1 (K): now also R39.1; no longer R17.1
- new net: R2.2, R5.1, U1.3 (+)
- new net: R33.2, R36.1, U4.13 (-)
- new net: R36.2, SW3.3 (C), U4.14
- new net: R30.2, R35.1, U3.7
- new net: R21.1, R22.2, U5.13 (-)
- new net: D2.1 (K), R8.1
- new net: D2.2 (A), SW2.5 (B)
- new net: R25.2, R26.2, R28.1, R30.1, U3.6 (-)
- new net: R25.1, RV3.2
- new net: Q2.1 (E1), Q2.4 (E2), R41.1
- new net: J3.T, R24.1
- new net: J4.T, R26.1
- new net: Q4.1 (B), Q5.1 (B), R40.1, SW3.2 (B)
- new net: Q4.2 (E), Q5.2 (E), R39.2
- new net: J6.T, R40.2
- new net: R33.1, RV4.1, SW3.1 (A), U4.8
- new net: Q3.1 (E1), Q3.4 (E2), R42.1
- new net: R29.2, R34.1, U3.1
- new net: R23.2, R24.2, R27.1, R29.1, U3.2 (-)
- new net: R31.2, RV4.2, RV4.3, U4.9 (-)
- new net I_ABC: Q2.6 (C1), Q3.6 (C1), U5.16
- no-connect marks 7 -> 13
Other:
- moved on the sheet: C1, C2, C3, C4, C5, C6, D3, D4, D6, H1
