File: lib/kicad/cynthia.kicad_blocks/Eurorack 10-pin header.kicad_block/Eurorack 10-pin header.kicad_sch (KiCad schematic)
At the start: 5 parts

Commit message: added 05
Parts:
- removed D11, D12: SS14, Diode_SMD:D_SMA, symbol Diode:SS14
- added D1, D2: 1N5819HW-7-F, Diode_SMD:D_SOD-123, symbol Diode:1N5819WS
Connections:
- net -12V: now also D1.2 (A)
- net at H1.1 (Pin_1), H1.2 (Pin_2): now also D2.2 (A)
- net at H1.10 (Pin_10), H1.9 (Pin_9): now also D1.1 (K)
Other:
- moved on the sheet: C1, C2, H1
