File: 05_midi_to_cv/05_midi_to_cv_conductor.kicad_pcb (KiCad board)
At the start: 2 copper layers, 40 x 100 mm, 33 parts, among them IC1 TLP2662, IC2 TLP2662, IC3 TLP2662, J1 MIDI IN 1, J2 MIDI IN 2, J3 MIDI IN 3, J4 AudioJack2, J5 Midi Fast Bus, J6 AudioJack2, J7 AudioJack2, U1 NCP1117-5.0_SOT223, U2 SN74HCT125

Commit message: updated 05
Parts:
- C1, C2, C5, C6, D1, D2: moved to F.Cu
- J4, J6, J7: value AudioJack2 -> ~; footprint cynthia:3.5mm jack mono -> cynthia:3.5mm thonk jack socket mono switched
- moved C1 50.1 mm to (58.3, 91.8), turned to 0 degrees
- moved C2 42.5 mm to (51.2, 91.8)
- moved J5 38.7 mm to (56.6, 39.6), turned to 0 degrees
- moved D2 37.8 mm to (51.0, 73.8), turned to 90 degrees
- moved H1 33.3 mm to (56.1, 72.5)
- moved D1 28.5 mm to (51.0, 83.8), turned to -90 degrees
- moved C9 20.1 mm to (40.8, 89.2), turned to -90 degrees
- moved U2 19.6 mm to (35.5, 92.2)
- moved R7 16.9 mm to (27.0, 98.5), turned to 180 degrees
- moved J4 12.8 mm to (30.7, 102.0), turned to -90 degrees
- moved R2 11.9 mm to (36.2, 105.5)
- moved J6 11.8 mm to (30.5, 114.2), turned to -90 degrees
- moved R4 11.1 mm to (36.0, 117.8)
- moved R6 10.8 mm to (36.0, 130.5)
- moved C8 10.4 mm to (36.2, 123.5), turned to 180 degrees
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Routing:
- net +3.3V: track 0.00 -> 105.0 mm
- net /midi input2/MIDI_IN: track 0.00 -> 101.6 mm
- net +5V: track 0.00 -> 88.5 mm, vias 0 -> 4
- net /midi input1/MIDI_IN: track 0.00 -> 83.7 mm, vias 0 -> 4
- net /midi input/MIDI_IN: track 0.00 -> 72.2 mm, vias 0 -> 4
- net +12V: track 0.00 -> 62.2 mm
- net -12V: track 0.00 -> 55.2 mm
- net MIDI_BUS: track 0.00 -> 46.2 mm, vias 0 -> 2
- net Net-(R9-Pad1): track 0.00 -> 34.4 mm
- net RUN: track 0.00 -> 28.9 mm
- net CLOCK: track 0.00 -> 27.6 mm
- net RESET: track 0.00 -> 26.0 mm
- net Net-(IC3-Pad1): track 0.00 -> 20.8 mm
- net Net-(IC1-Pad1): track 0.00 -> 20.5 mm
- net Net-(IC2-Pad1): track 0.00 -> 20.5 mm
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- added copper zone on F.Cu, net +5V
- added copper zone on B.Cu, net GND

Commit message: dual board 05
Parts:
- removed C8: 100nF, cynthia:C SMD 0805
- added C4: 100nF, cynthia:C SMD 0805, F.Cu at (121.5, 70.5)
- added J10: ui top, Connector_PinHeader_2.54mm:PinHeader_1x08_P2.54mm_Vertical, B.Cu at (90.0, 106.0)
- added J11: main top, Connector_PinSocket_2.54mm:PinSocket_1x08_P2.54mm_Vertical, F.Cu at (116.0, 106.0)
- added J8: ui_top, Connector_PinHeader_2.54mm:PinHeader_1x04_P2.54mm_Vertical, B.Cu at (88.2, 147.0)
- added J9: main_top, Connector_PinSocket_2.54mm:PinSocket_1x04_P2.54mm_Vertical, F.Cu at (114.2, 147.0)
- A1: footprint Module:RaspberryPi_Pico_Common_Unspecified -> Module:RaspberryPi_Pico_SMD_HandSolder; moved to B.Cu
- moved C3 107.0 mm to (133.5, 53.5)
- moved R2 105.5 mm to (128.0, 53.5)
- moved R6 101.6 mm to (128.0, 87.5)
- moved C7 100.0 mm to (133.5, 87.5)
- moved R7 99.7 mm to (126.0, 110.0), turned to -90 degrees
- moved R9 97.4 mm to (123.5, 110.0), turned to -90 degrees
- moved IC1 94.8 mm to (130.0, 60.0), turned to 0 degrees
- moved J6 94.7 mm to (124.0, 129.0)
- moved J7 94.6 mm to (124.0, 141.5)
- moved J4 94.5 mm to (124.0, 117.0)
- moved R8 94.0 mm to (121.0, 110.0), turned to -90 degrees
- moved R4 92.9 mm to (116.0, 70.5)
- moved IC3 91.4 mm to (130.0, 94.0), turned to 0 degrees
- moved J5 89.2 mm to (92.0, 121.5), turned to 180 degrees
- moved H1 86.7 mm to (105.8, 143.6), turned to 180 degrees
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Connections:
- net /midi input/MIDI_IN renamed MIDI_1
- net /midi input/MIDI_IN_RING renamed Net-(J1-PadR)
- net /midi input/MIDI_IN_TIP renamed Net-(IC1-Pad2)
- net /midi input1/MIDI_IN renamed MIDI_2
- net /midi input1/MIDI_IN_RING renamed Net-(J2-PadR)
- net /midi input1/MIDI_IN_TIP renamed Net-(IC2-Pad2)
- net /midi input2/MIDI_IN renamed MIDI_3
- net /midi input2/MIDI_IN_RING renamed Net-(J3-PadR)
- net /midi input2/MIDI_IN_TIP renamed Net-(IC3-Pad2)
- net MIDI_BUS renamed Net-(A1-GPIO16)
- A1 pad 24: RESET -> Net-(A1-GPIO18)
- A1 pad 25: RUN -> Net-(A1-GPIO19)
- A1 pad 26: CLOCK -> Net-(A1-GPIO20)
- R7 pad 1: Net-(R7-Pad1) -> CLOCK
- R8 pad 1: Net-(R8-Pad1) -> RUN
- R9 pad 1: Net-(R9-Pad1) -> RESET
- U2 pad 2: CLOCK -> Net-(A1-GPIO20)
- U2 pad 3: Net-(R7-Pad1) -> CLOCK
- U2 pad 5: RUN -> Net-(A1-GPIO19)
- U2 pad 6: Net-(R8-Pad1) -> RUN
- U2 pad 8: Net-(R9-Pad1) -> RESET
- U2 pad 9: RESET -> Net-(A1-GPIO18)
Routing:
- net +3.3V: track 105.0 -> 199.4 mm, vias 0 -> 5
- net MIDI_1: track 72.2 -> 122.9 mm, vias 4 -> 1
- net MIDI_3: track 101.6 -> 59.1 mm, vias 0 -> 1
- net -12V: track 55.2 -> 19.8 mm
- net Net-(R9-Pad1): track 34.4 -> 0.00 mm
- net Net-(J7-PadT): track 3.56 -> 34.7 mm
- net Net-(A1-GPIO16): track 46.2 -> 17.6 mm, vias 2 -> 1
- net GND: track 15.8 -> 42.7 mm, vias 13 -> 10
- net Net-(R8-Pad1): track 19.5 -> 0.00 mm
- net MIDI_2: track 83.7 -> 101.8 mm, vias 4 -> 3
- net +12V: track 62.2 -> 45.5 mm
- net Net-(J6-PadT): track 3.54 -> 19.8 mm
- net Net-(J3-PadR): track 3.95 -> 18.1 mm
- net Net-(A1-GPIO18): track 0.00 -> 14.2 mm, vias 0 -> 1
- net Net-(J1-PadR): track 3.95 -> 17.6 mm
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Other:
- board size 40 x 100 mm -> 52 x 100 mm
