File: 05_midi_to_cv/midi_input.kicad_sch (KiCad schematic)
At the start: 4 parts, among them IC1 TLP2662

Commit message: dual board 05
Parts:
- removed C3: 100nF, cynthia:C SMD 0805, symbol Device:C
- removed IC1: TLP2662, Package_DIP:SMDIP-8_W7.62mm, symbol cynthia:TLP2662
- removed R1: 100R, cynthia:R SMD 0805, symbol Device:R
- removed R2: 4.7k, cynthia:R SMD 0805, symbol Device:R
