File: 05_midi_to_cv/conductor/05_midi_to_cv_conductor.kicad_pcb (KiCad board)
At the start: 2 copper layers, 52 x 100 mm, 37 parts, among them IC1 TLP2662, IC2 TLP2662, IC3 TLP2662, J1 MIDI IN 1, J10 ui top, J11 main top, J2 MIDI IN 2, J3 MIDI IN 3, J5 Midi Fast Bus, J8 ui_top, J9 main_top, U1 NCP1117-5.0_SOT223, U2 SN74HCT125

Commit message: moved conductor
Parts:
- moved C1 110.4 mm to (5.50, 73.0)
- moved C2 110.4 mm to (3.32, 66.0)
- moved D1 110.4 mm to (10.1, 66.0)
- moved D2 110.4 mm to (9.82, 73.0)
- moved A1 98.7 mm to (12.9, 26.5)
- moved C3 98.6 mm to (48.5, 3.50)
- moved C4 98.6 mm to (36.5, 20.5)
- moved C5 98.6 mm to (13.5, 63.0)
- moved C6 98.6 mm to (20.5, 63.0)
- moved C7 98.6 mm to (48.5, 37.5)
- moved C9 98.6 mm to (15.5, 34.5)
- moved H1 98.6 mm to (20.8, 93.6)
- moved IC1 98.6 mm to (45.0, 10.0)
- moved IC2 98.6 mm to (33.0, 27.0)
- moved IC3 98.6 mm to (45.0, 44.0)
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Routing:
- net Net-(A1-GPIO16): track 17.6 -> 37.2 mm
- net Net-(D2-A): track 8.97 -> 26.2 mm
- net Net-(D1-K): track 7.85 -> 22.9 mm
- net -12V: track 19.8 -> 27.5 mm
- net +12V: track 45.5 -> 41.6 mm
