File: lib/kicad/cynthia.kicad_blocks/eurorack 10pin header.kicad_block/eurorack 10pin header.kicad_sch (KiCad schematic)
At the start: 5 parts

Commit message: fine-tuned 05
Parts:
- C1, C2: footprint Capacitor_THT:CP_Radial_D6.3mm_P2.50mm -> cynthia:CP_Radial_D6.3mm_P2.50mm; KiLib_Generator (none) -> capacitor/THT/other
- H1: KiLib_Generator (none) -> connector/pin_header_socket
Connections:
- net +12V: now also D2.1 (K)
Other:
- moved on the sheet: C1, C2, D1, H1
