File: 05_midi_to_cv/conductor/conductor_controls/conductor_controls.kicad_sch (KiCad schematic)
At the start: 23 parts, among them IC1 TLP2662, IC2 TLP2662, IC3 TLP2662, J1 MIDI IN 1, J2 MIDI IN 2, J3 MIDI IN 3, U2 SN74HCT125

Commit message: fine-tuned 05
Parts:
- removed C9: 100nF, cynthia:C SMD 0805, symbol Device:C
- removed J1: MIDI IN 1, cynthia:3.5mm jack stereo, symbol Connector_Audio:AudioJack3
- removed J2: MIDI IN 2, cynthia:3.5mm jack stereo, symbol Connector_Audio:AudioJack3
- removed J3: MIDI IN 3, cynthia:3.5mm jack stereo, symbol Connector_Audio:AudioJack3
- removed J4, J6, J7: (no value), cynthia:3.5mm thonk jack socket mono switched, symbol cynthia:3.5mm thonk jack socket mono switched
- removed U2: SN74HCT125, Package_SO:SOIC-14_3.9x8.7mm_P1.27mm, symbol 74xx:74AHCT125
- added J1, J2, J3: (no value), cynthia:3.5mm jack stereo round, symbol cynthia:3.5mm jack stereo
- added J4: to main board, Connector_PinSocket_2.54mm:PinSocket_1x08_P2.54mm_Vertical, symbol Connector:Conn_01x08_Socket
- added J5, J6, J7: (no value), cynthia:3.5mm thonk jack socket mono switched, symbol cynthia:3.5mm jack mono switched
- added J9: Conn_01x04_Socket, Connector_PinSocket_2.54mm:PinSocket_1x04_P2.54mm_Vertical, symbol Connector:Conn_01x04_Socket
- renumbered C3 to C1, C4 to C2, C7 to C3, R3 to R2, R5 to R3, R2 to R4, R4 to R5
Connections:
- net +3.3V: now also J4.1 (Pin_1)
- net CLOCK: now also J4.5 (Pin_5)
- net GND: now also J4.2 (Pin_2), J5.S, J6.S, J7.S, J9.1 (Pin_1), J9.2 (Pin_2), J9.3 (Pin_3), J9.4 (Pin_4)
- net MIDI_1: now also J4.6 (Pin_6)
- net MIDI_2: now also J4.7 (Pin_7)
- net MIDI_3: now also J4.8 (Pin_8)
- net RESET: now also J4.4 (Pin_4)
- net RUN: now also J4.3 (Pin_3)
- net at R2.1: now also J2.R
- net at R3.1: now also J3.R
- net at R1.1: now also J1.R
- net at IC1.2, IC1.4: now also J1.T
- net at R8.2: now also J6.T
- net at IC3.2, IC3.4: now also J3.T
- net at R7.2: now also J5.T
- net at IC2.2, IC2.4: now also J2.T
- net at R9.2: now also J7.T
Other:
- title: (none) -> conductor control board
- moved on the sheet: R2

Commit message: worked on issues after building #05
Parts:
- IC1, IC2, IC3: footprint Package_DIP:SMDIP-8_W7.62mm -> cynthia:SMDIP-8_W7.62mm_hand_solder
Other:
- title: conductor control board -> #05: Conductor - Control Board
Changed lines of the file:
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@@
 	(paper "A4")
 	(title_block
-		(title "conductor control board")
-		(date "2026-09-19")
-		(rev "0.1")
+		(title "#05: Conductor - Control Board")
+		(date "2026-10-24")
+		(rev "2")
 	)
 	(junction
@@
 			)
 		)
-		(property "Footprint" "Package_DIP:SMDIP-8_W7.62mm"
+		(property "Footprint" "cynthia:SMDIP-8_W7.62mm_hand_solder"
 			(at 71.12 55.88 0)
 			(hide yes)
@@
 			)
 		)
-		(property "Footprint" "Package_DIP:SMDIP-8_W7.62mm"
+		(property "Footprint" "cynthia:SMDIP-8_W7.62mm_hand_solder"
 			(at 71.12 96.52 0)
 			(hide yes)
@@
 			)
 		)
-		(property "Footprint" "Package_DIP:SMDIP-8_W7.62mm"
+		(property "Footprint" "cynthia:SMDIP-8_W7.62mm_hand_solder"
 			(at 71.12 137.16 0)
 			(hide yes)
