File: 05_midi_to_cv/conductor/conductor_main/conductor_main.kicad_pcb (KiCad board)
At the start: 2 copper layers, 26 x 100 mm, 14 parts, among them J1 ui_top, J2 Midi Fast Bus, J3 ui top, U1 SN74HCT125, U2 NCP1117-5.0_SOT223

Commit message: worked on issues after building #05
Parts:
- U1: footprint Package_SO:SOIC-14_3.9x8.7mm_P1.27mm -> cynthia:SOIC-14_3.9x8.7mm_P1.27mm
Routing:
- net CLOCK: track 20.9 -> 21.9 mm
- net +5V: track 75.2 -> 76.0 mm
Other:
- board text added: "#05: Conductor: Main Board Rev. 2 2026 Benjamin Murauer"
