File: 05_midi_to_cv/conductor/conductor_main/conductor_main.kicad_sch (KiCad schematic)
At the start: 15 parts, among them J10 ui top, J11 main top, J5 Midi Fast Bus, J8 ui_top, J9 main_top, U1 NCP1117-5.0_SOT223, U2 SN74HCT125

Commit message: fine-tuned 05
Parts:
- removed J11: main top, Connector_PinSocket_2.54mm:PinSocket_1x08_P2.54mm_Vertical, symbol Connector:Conn_01x08_Socket
- removed J9: main_top, Connector_PinSocket_2.54mm:PinSocket_1x04_P2.54mm_Vertical, symbol Connector:Conn_01x04_Socket
- added C2: 100nF, cynthia:C SMD 0805, symbol Device:C
- added unit 5 of U1
- A1: footprint Module:RaspberryPi_Pico_SMD_HandSolder -> Module:RaspberryPi_Pico_Common_Unspecified
- D1: renamed from D2; footprint Diode_SMD:D_SOD-323 -> Diode_SMD:D_SOD-123
- D2: renamed from D1; footprint Diode_SMD:D_SOD-323 -> Diode_SMD:D_SOD-123
- renumbered C5 to C1, C6 to C3, C1 to C4, C2 to C5, J8 to J1, J5 to J2, J10 to J3, U2 to U1, U1 to U2
Connections:
- net +3.3V: now also J3.1 (Pin_1); no longer J3.2 (Pin_2)
- net +5V: now also C2.1, U1.14 (VCC); no longer J3.1 (Pin_1)
- net GND: now also J3.2 (Pin_2), C2.2, U1.7 (GND); no longer A1.33 (AGND)
- no-connect marks 26 -> 27
Other:
- removed sheet ui

Commit message: finished firmware for 05 melodic player
Other:
- moved on the sheet: J1
Changed lines of the file:
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@@
 	(paper "A4")
 	(junction
-		(at 104.14 58.42)
+		(at 30.48 34.29)
 		(diameter 0)
 		(color 0 0 0 0)
@@
 	)
 	(junction
-		(at 104.14 55.88)
+		(at 30.48 31.75)
 		(diameter 0)
 		(color 0 0 0 0)
@@
 	)
 	(junction
-		(at 104.14 53.34)
+		(at 30.48 29.21)
 		(diameter 0)
 		(color 0 0 0 0)
@@
 	(wire
 		(pts
-			(xy 104.14 58.42) (xy 104.14 62.23)
+			(xy 30.48 34.29) (xy 30.48 38.1)
 		)
 		(stroke
@@
 	(wire
 		(pts
-			(xy 104.14 50.8) (xy 104.14 53.34)
+			(xy 30.48 26.67) (xy 30.48 29.21)
 		)
 		(stroke
@@
 	(wire
 		(pts
-			(xy 101.6 53.34) (xy 104.14 53.34)
+			(xy 27.94 29.21) (xy 30.48 29.21)
 		)
 		(stroke
@@
 	(wire
 		(pts
-			(xy 101.6 50.8) (xy 104.14 50.8)
+			(xy 27.94 26.67) (xy 30.48 26.67)
 		)
 		(stroke
@@
 	(wire
 		(pts
-			(xy 104.14 53.34) (xy 104.14 58.42)
+			(xy 30.48 29.21) (xy 30.48 34.29)
 		)
 		(stroke
@@
 	(wire
 		(pts
-			(xy 101.6 55.88) (xy 104.14 55.88)
+			(xy 27.94 31.75) (xy 30.48 31.75)
 		)
 		(stroke
@@
 	(wire
 		(pts
-			(xy 101.6 58.42) (xy 104.14 58.42)
+			(xy 27.94 34.29) (xy 30.48 34.29)
 		)
 		(stroke
@@
 	)
 	(global_label "MIDI_2"
-		(shape input)
+		(shape output)
 		(at 147.32 86.36 0)
 		(fields_autoplaced yes)
@@
 	)
 	(global_label "MIDI_3"
-		(shape input)
+		(shape output)
 		(at 147.32 88.9 0)
 		(fields_autoplaced yes)
@@
 	)
 	(global_label "RUN"
-		(shape output)
+		(shape input)
 		(at 147.32 76.2 0)
 		(fields_autoplaced yes)
@@
 	)
 	(global_label "RESET"
-		(shape output)
+		(shape input)
 		(at 147.32 78.74 0)
 		(fields_autoplaced yes)
@@
 	)
 	(global_label "MIDI_1"
-		(shape input)
+		(shape output)
 		(at 147.32 83.82 0)
 		(fields_autoplaced yes)
@@
 	)
 	(global_label "CLOCK"
-		(shape output)
+		(shape input)
 		(at 147.32 81.28 0)
 		(fields_autoplaced yes)
@@
 	(symbol
 		(lib_id "power:GND")
-		(at 104.14 62.23 0)
+		(at 30.48 38.1 0)
 		(unit 1)
 		(body_style 1)
@@
 		(fields_autoplaced yes)
 		(property "Reference" "#PWR08"
-			(at 104.14 68.58 0)
+			(at 30.48 44.45 0)
 			(hide yes)
 			(show_name no)
@@
 		)
 		(property "Value" "GND"
-			(at 104.14 67.31 0)
+			(at 30.48 43.18 0)
 			(show_name no)
 			(do_not_autoplace no)
@@
 		)
 		(property "Footprint" "Module:RaspberryPi_Pico_Common_Unspecified"
-			(at 104.14 62.23 0)
+			(at 30.48 38.1 0)
 			(hide yes)
 			(show_name no)
@@
 		)
 		(property "Datasheet" ""
-			(at 104.14 62.23 0)
+			(at 30.48 38.1 0)
 			(hide yes)
 			(show_name no)
@@
 		)
 		(property "Description" "Power symbol creates a global label with name \"GND\" , ground"
-			(at 104.14 62.23 0)
+			(at 30.48 38.1 0)
 			(hide yes)
 			(show_name no)
@@
 	(symbol
 		(lib_id "Connector:Conn_01x04_Pin")
-		(at 96.52 53.34 0)
+		(at 22.86 29.21 0)
 		(unit 1)
 		(body_style 1)
@@
 		(fields_autoplaced yes)
 		(property "Reference" "J1"
-			(at 97.155 45.72 0)
+			(at 23.495 21.59 0)
 			(show_name no)
 			(do_not_autoplace no)
@@
 		)
 		(property "Value" "ui_top"
-			(at 97.155 48.26 0)
+			(at 23.495 24.13 0)
 			(show_name no)
 			(do_not_autoplace no)
@@
 		)
 		(property "Footprint" "Connector_PinHeader_2.54mm:PinHeader_1x04_P2.54mm_Vertical"
-			(at 96.52 53.34 0)
+			(at 22.86 29.21 0)
 			(hide yes)
 			(show_name no)
@@
 		)
 		(property "Datasheet" ""
-			(at 96.52 53.34 0)
+			(at 22.86 29.21 0)
 			(hide yes)
 			(show_name no)
@@
 		)
 		(property "Description" "Generic connector, single row, 01x04, script generated"
-			(at 96.52 53.34 0)
+			(at 22.86 29.21 0)
 			(hide yes)
 			(show_name no)

Commit message: worked on issues after building #05
Parts:
- U1: footprint Package_SO:SOIC-14_3.9x8.7mm_P1.27mm -> cynthia:SOIC-14_3.9x8.7mm_P1.27mm
Other:
- title: (none) -> #05: Conductor: Main Board
Changed lines of the file:
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@@
 	(generator_version "10.0")
 	(paper "A4")
+	(title_block
+		(title "#05: Conductor: Main Board")
+		(date "2026-10-24")
+		(rev "2")
+	)
 	(junction
 		(at 30.48 34.29)
@@
 			)
 		)
-		(property "Footprint" "Package_SO:SOIC-14_3.9x8.7mm_P1.27mm"
+		(property "Footprint" "cynthia:SOIC-14_3.9x8.7mm_P1.27mm"
 			(at 106.68 172.72 0)
 			(hide yes)
@@
 			)
 		)
-		(property "Footprint" "Package_SO:SOIC-14_3.9x8.7mm_P1.27mm"
+		(property "Footprint" "cynthia:SOIC-14_3.9x8.7mm_P1.27mm"
 			(at 30.48 181.61 0)
 			(hide yes)
@@
 			)
 		)
-		(property "Footprint" "Package_SO:SOIC-14_3.9x8.7mm_P1.27mm"
+		(property "Footprint" "cynthia:SOIC-14_3.9x8.7mm_P1.27mm"
 			(at 139.7 177.8 0)
 			(hide yes)
@@
 			)
 		)
-		(property "Footprint" "Package_SO:SOIC-14_3.9x8.7mm_P1.27mm"
+		(property "Footprint" "cynthia:SOIC-14_3.9x8.7mm_P1.27mm"
 			(at 106.68 132.08 0)
 			(hide yes)
@@
 			)
 		)
-		(property "Footprint" "Package_SO:SOIC-14_3.9x8.7mm_P1.27mm"
+		(property "Footprint" "cynthia:SOIC-14_3.9x8.7mm_P1.27mm"
 			(at 106.68 152.4 0)
 			(hide yes)
