File: 05_midi_to_cv/player_drum_velocity/player_drum_velocity.kicad_pcb (KiCad board)
At the start: 2 copper layers, 18 x 100 mm, 31 parts, among them J1 SWD header, J5 Midi Fast Bus, Q1 BC847, Q2 BC847, SW1 SW_Push, SW2 SW_Push, U1 STM32G030F6Px, U2 MCP1700x-330xxTT, U3 NCP1117-5.0_SOT223, U4 MCP4822, U5 TL072

Commit message: fine-tuned 05
Parts:
- moved J6 58.5 mm to (9.00, 94.5)
- moved J4 57.7 mm to (9.00, 83.7)
- moved Q2 57.7 mm to (9.00, 83.7)
- moved R3 57.7 mm to (14.5, 87.2)
- moved R4 57.7 mm to (5.50, 87.2)
- moved R6 57.7 mm to (2.00, 84.7)
- moved R8 56.5 mm to (2.00, 93.5), turned to 90 degrees
- moved C6 20.8 mm to (11.5, 59.2)
- moved SW2 20.8 mm to (15.7, 54.3)
- moved C1 20.8 mm to (6.25, 24.2)
- moved C2 20.8 mm to (15.8, 23.0)
- moved C3 20.8 mm to (11.2, 45.8)
- moved C4 20.8 mm to (3.96, 75.2)
- moved C5 20.8 mm to (12.5, 75.2)
- moved C7 20.8 mm to (15.0, 56.2)
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- renumbered C9 to C1, C10 to C2, C8 to C3, C5 to C4, C6 to C5, C7 to C6, C4 to C7, C1 to C8, J5 to J1, J1 to J2, J2 to J3, J6 to J4, J4 to J5, J3 to J6, R8 to R1, R9 to R2, R12 to R3, R13 to R4, R10 to R5, R11 to R6, R6 to R7, R5 to R8, U5 to U1, U1 to U2, U2 to U4, U4 to U5
Routing:
- net Net-(U1B--): track 10.1 -> 76.7 mm, vias 0 -> 2
- net Net-(U2-PA2): track 56.1 -> 35.6 mm
- net Net-(U1A--): track 34.2 -> 15.3 mm
- net GND: track 37.9 -> 27.0 mm, vias 8 -> 10
- net Net-(U2-PA3): track 36.0 -> 45.4 mm
- net +5V: track 99.8 -> 94.3 mm, vias 2 -> 1
- net Net-(Q2-C): track 8.13 -> 11.0 mm

Commit message: updated drum velocity
Parts:
- removed SW2: SW_Push, Button_Switch_THT:SW_PUSH_6mm_H8.5mm
- added D1: LED, LED_THT:LED_D5.0mm, B.Cu at (12.2, 51.2)
- added R9: 4.7k, cynthia:R SMD 0805, F.Cu at (9.00, 51.2)
- moved SW1 0.25 mm to (7.50, 54.5)
Routing:
- net Net-(D1-A): track 11.1 -> 7.70 mm
- net Net-(D1-K): track 0.00 -> 2.22 mm
- net GND: track 27.0 -> 25.2 mm, vias 10 -> 13
- net Net-(U2-PA0): track 15.8 -> 16.7 mm

Commit message: 05 rev1
Parts:
- moved J3 0.55 mm to (9.00, 5.50)
- moved J5 0.50 mm to (9.00, 16.5)
- moved D1 0.28 mm to (12.5, 51.2)
- moved J4 0.20 mm to (9.00, 83.5)
Changed lines of the file:
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@@
 			(outputformat 1)
 			(mirror no)
-			(drillshape 1)
+			(drillshape 0)
 			(scaleselection 1)
-			(outputdirectory "")
+			(outputdirectory "./")
 		)
 	)
@@
 			)
 		)
-		(property "Description" "LEARN 1"
+		(property "Description" "LEARN"
 			(at 0 0 270)
 			(unlocked yes)
@@
 	(footprint "cynthia:3.5mm thonk jack socket mono switched"
 		(layer "B.Cu")
-		(at 9 83.7 -90)
+		(at 9 83.5 -90)
 		(property "Reference" "J4"
 			(at -2.54 -8.382 90)
@@
 	(footprint "LED_THT:LED_D5.0mm"
 		(layer "B.Cu")
-		(at 12.225 51.25)
+		(at 12.5 51.25)
 		(descr "LED, diameter 5.0mm, 2 pins, http://cdn-reichelt.de/documents/datenblatt/A500/LL-504BC2E-009.pdf, generated by kicad-footprint-generator")
 		(tags "LED")
@@
 		)
 		(point
-			(at 13.495 51.25)
+			(at 13.77 51.25)
 			(size 2)
 			(layer "B.Fab")
@@
 	(footprint "cynthia:3.5mm thonk jack socket mono switched"
 		(layer "B.Cu")
-		(at 9 16 -90)
+		(at 9 16.5 -90)
 		(property "Reference" "J5"
 			(at -2.54 -8.382 90)
@@
 	(footprint "cynthia:3.5mm thonk jack socket mono switched"
 		(layer "B.Cu")
-		(at 9 6.05 -90)
+		(at 9 5.5 -90)
 		(property "Reference" "J3"
 			(at -2.54 -8.382 90)
@@
 	)
 	(segment
-		(start 13.9625 56.25)
-		(end 13.9625 53.75)
+		(start 13.9625 53.75)
+		(end 13.9625 56.25)
+		(width 0.2)
+		(layer "F.Cu")
+		(net "+3.3V")
+	)
+	(segment
+		(start 12.2875 45.75)
+		(end 13.75 47.2125)
+		(width 0.2)
+		(layer "F.Cu")
+		(net "+3.3V")
+	)
+	(segment
+		(start 13.75 47.2125)
+		(end 13.75 53.5375)
 		(width 0.2)
 		(layer "F.Cu")
@@
 	)
 	(segment
-		(start 13.425 46.8875)
-		(end 13.425 53.2125)
+		(start 13.75 53.5375)
+		(end 13.9625 53.75)
 		(width 0.2)
 		(layer "F.Cu")
@@
 	)
 	(segment
-		(start 13.425 53.2125)
-		(end 13.9625 53.75)
-		(width 0.2)
-		(layer "F.Cu")
-		(net "+3.3V")
-	)
-	(segment
-		(start 12.2875 45.75)
-		(end 13.425 46.8875)
-		(width 0.2)
-		(layer "F.Cu")
-		(net "+3.3V")
-	)
-	(segment
 		(start 6.315 35.755)
 		(end 4.23 33.67)
@@
 	)
 	(segment
-		(start 13.475 25.405)
-		(end 13.475 24.135)
+		(start 8.795552 20.25)
+		(end 4.25 20.25)
 		(width 0.2)
 		(layer "F.Cu")
@@
 	(segment
 		(start 12.680552 24.135)
-		(end 6.545552 18)
+		(end 8.795552 20.25)
 		(width 0.2)
 		(layer "F.Cu")
@@
 	)
 	(segment
-		(start 6.545552 18)
-		(end 2 18)
+		(start 13.475 25.405)
+		(end 13.475 24.135)
 		(width 0.2)
 		(layer "F.Cu")
@@
 	)
 	(segment
+		(start 4.25 20.25)
+		(end 2 18)
+		(width 0.2)
+		(layer "F.Cu")
+		(net "Net-(U1A--)")
+	)
+	(segment
 		(start 17 28.595)
 		(end 17 23.690256)
@@
 	)
 	(segment
+		(start 14.765 51.25)
+		(end 14.765 43.7525)
+		(width 0.2)
+		(layer "F.Cu")
+		(net "Net-(D1-A)")
+	)
+	(segment
+		(start 14.765 43.7525)
+		(end 14.625 43.6125)
+		(width 0.2)
+		(layer "F.Cu")
+		(net "Net-(D1-A)")
+	)
+	(segment
 		(start 15.925 43.6125)
 		(end 17 44.6875)
@@
 	)
 	(segment
-		(start 2 6.05)
-		(end 4.6 6.05)
-		(width 0.2)
-		(layer "F.Cu")
-		(net "Net-(J3-PadT)")
-	)
-	(segment
 		(start 12.225 51.25)
 		(end 10 51.25)
@@
 	)
 	(segment
-		(start 14.765 51.25)
-		(end 14.765 43.7525)
-		(width 0.2)
-		(layer "F.Cu")
-		(net "Net-(D1-A)")
-	)
-	(segment
-		(start 14.765 43.7525)
-		(end 14.625 43.6125)
+		(start 2 6.05)
+		(end 4.6 6.05)
 		(width 0.2)
 		(layer "F.Cu")
-		(net "Net-(D1-A)")
+		(net "Net-(J3-PadT)")
 	)
 	(zone

Commit message: worked on issues after building #05
Parts:
- added R10: 10k, cynthia:R SMD 0805, F.Cu at (134.2, 54.8)
- added R11: 10k, cynthia:R SMD 0805, F.Cu at (127.0, 65.0)
- added R12: 15k, cynthia:R SMD 0805, F.Cu at (134.2, 57.0)
- added R13: 15k, cynthia:R SMD 0805, F.Cu at (127.0, 61.0)
- R9: value 4.7k -> 2.2k
- U5: footprint Package_SO:SOIC-8_5.3x6.2mm_P1.27mm -> cynthia:SOIC-8_3.9x4.9mm_P1.27mm
- moved C1 138.9 mm to (140.5, 60.0)
- moved C3 131.2 mm to (136.2, 85.8)
- moved C4 131.2 mm to (129.0, 115.2)
- moved C5 131.2 mm to (137.5, 115.2)
- moved C6 131.2 mm to (136.5, 99.2)
- moved C7 131.2 mm to (140.0, 96.2)
- moved C8 131.2 mm to (130.8, 68.5)
- moved D1 131.2 mm to (137.5, 91.2)
- moved J1 131.2 mm to (131.5, 109.2)
- moved J2 131.2 mm to (129.2, 73.7)
- moved J3 131.2 mm to (134.0, 45.5)
- moved J4 131.2 mm to (134.0, 123.5)
- moved J5 131.2 mm to (134.0, 56.5)
- moved J6 131.2 mm to (134.0, 134.5)
- moved Q1 131.2 mm to (134.0, 46.0)
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Connections:
- R7 pad 2: Net-(U1A--) -> Net-(R13-Pad1)
- R8 pad 2: Net-(U1B--) -> Net-(R12-Pad1)
- U1 pad 1: Net-(U1A--) -> Net-(R13-Pad1)
- U1 pad 7: Net-(U1B--) -> Net-(R12-Pad1)
Routing:
- net Net-(R12-Pad1): track 0.00 -> 84.8 mm, vias 0 -> 2
- net Net-(U1B--): track 76.7 -> 10.9 mm
- net +12V: track 80.0 -> 92.0 mm, vias 0 -> 2
- net GND: track 25.2 -> 35.5 mm
- net -12V: track 61.9 -> 52.3 mm, vias 2 -> 0
- net Net-(R13-Pad1): track 0.00 -> 8.60 mm
- net Net-(U1A--): track 15.3 -> 7.58 mm
- net Net-(U1B-+): track 14.8 -> 10.1 mm
- net Net-(U1A-+): track 10.2 -> 11.5 mm, vias 0 -> 2
- net Net-(U2-PA4): track 11.2 -> 12.4 mm
- net +5V: track 94.3 -> 93.4 mm
- net Net-(U2-PA5): track 10.00 -> 10.5 mm
Other:
- board text added: "#05: Drum Velocity Player Rev. 2 2026 Benjamin Murauer"
