File: 05_midi_to_cv/player_drum_velocity/player_drum_velocity.kicad_sch (KiCad schematic)
At the start: 31 parts, among them J1 SWD header, J5 Midi Fast Bus, Q1 BC847, Q2 BC847, SW1 SW_Push, SW2 SW_Push, U1 STM32G030F6Px, U2 MCP1700x-330xxTT, U3 NCP1117-5.0_SOT223, U4 MCP4822, U5 TL072

Commit message: fine-tuned 05
Parts:
- J3: renamed from J2; symbol cynthia:3.5mm thonk jack socket mono switched -> cynthia:3.5mm jack mono switched
- J4: renamed from J6; symbol cynthia:3.5mm thonk jack socket mono switched -> cynthia:3.5mm jack mono switched
- J5: renamed from J4; symbol cynthia:3.5mm thonk jack socket mono switched -> cynthia:3.5mm jack mono switched
- J6: renamed from J3; symbol cynthia:3.5mm thonk jack socket mono switched -> cynthia:3.5mm jack mono switched
- renumbered C9 to C1, C10 to C2, C8 to C3, C5 to C4, C6 to C5, C7 to C6, C4 to C7, C1 to C8, J5 to J1, J1 to J2, R8 to R1, R9 to R2, R12 to R3, R13 to R4, R10 to R5, R11 to R6, R6 to R7, R5 to R8, U5 to U1, U1 to U2, U2 to U4, U4 to U5

Commit message: updated drum velocity
Parts:
- removed SW2: SW_Push, Button_Switch_THT:SW_PUSH_6mm_H8.5mm, symbol Switch:SW_Push
- added D1: LED, LED_THT:LED_D5.0mm, symbol Device:LED
- added R9: 4.7k, cynthia:R SMD 0805, symbol Device:R
Connections:
- net GND: now also R9.1
- net at U2.8 (PA1): now also D1.2 (A)
- new net: D1.1 (K), R9.2
- no-connect marks 13 -> 12

Commit message: 05 rev1
Changed lines of the file:
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@@
 			)
 		)
-		(property "Description" "LEARN 1"
+		(property "Description" "LEARN"
 			(at 99.06 74.676 0)
 			(show_name no)

Commit message: worked on issues after building #05
Parts:
- added R10, R11: 10k, cynthia:R SMD 0805, symbol Device:R
- added R12, R13: 15k, cynthia:R SMD 0805, symbol Device:R
- R9: value 4.7k -> 2.2k
- U5: footprint Package_SO:SOIC-8_5.3x6.2mm_P1.27mm -> cynthia:SOIC-8_3.9x4.9mm_P1.27mm
Connections:
- net GND: now also R10.1, R11.1
- net at R7.2, U1.1: now also R13.1; no longer U1.2 (-)
- net at R8.2, U1.7: now also R12.1; no longer U1.6 (-)
- new net: R11.2, R13.2, U1.2 (-)
- new net: R10.2, R12.2, U1.6 (-)
Other:
- title: (none) -> #02 Player: Double Drums with Velocity
