File: 05_midi_to_cv/player_melodic/player_melodic.kicad_pcb (KiCad board)
At the start: 2 copper layers, 18 x 100 mm, 27 parts, among them J1 SWD header, J5 Midi Fast Bus, Q1 BC847, SW1 SW_Push, U1 STM32G030F6Px, U2 MCP1700x-330xxTT, U3 NCP1117-5.0_SOT223, U4 MCP4822, U5 TL072

Commit message: fine-tuned 05
Parts:
- removed the J2 at (9.00, 26.0)
- removed R9: 10k, cynthia:R SMD 0805
- added J5: ~, cynthia:3.5mm thonk jack socket mono switched, B.Cu at (9.00, 16.0)
- added R2: 10k, cynthia:R SMD 0805, F.Cu at (9.50, 85.5)
- moved J3 78.2 mm to (9.00, 94.2)
- moved Q1 63.8 mm to (9.00, 94.2), turned to 180 degrees
- moved R4 61.6 mm to (5.25, 88.5), turned to 0 degrees
- moved R1 58.0 mm to (9.50, 88.5), turned to 0 degrees
- moved C1 12.8 mm to (15.0, 23.8)
- moved C2 12.8 mm to (8.00, 29.2)
- moved C3 12.8 mm to (13.0, 59.8)
- moved C5 12.8 mm to (9.00, 32.2)
- moved C7 12.8 mm to (11.5, 67.2)
- moved C8 12.8 mm to (16.0, 63.2)
- moved J1 12.8 mm to (4.98, 41.7)
- moved R3 12.8 mm to (4.50, 26.8)
- moved RV1 12.8 mm to (4.00, 33.8)
- moved SW1 12.8 mm to (7.50, 62.2)
- moved U1 12.8 mm to (13.0, 27.8)
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- renumbered C9 to C1, C10 to C2, C8 to C3, C5 to C4, C1 to C5, C4 to C8, J5 to J2, R8 to R1, R7 to R3, R10 to R4, R6 to R5, R5 to R6, U5 to U1, U1 to U2, U4 to U3, U3 to U4, U2 to U5
Connections:
- R4 pad 1: Net-(J2-PadT) -> Net-(J3-PadT)
- R6 pad 1: Net-(J3-PadT) -> Net-(J5-PadT)
Routing:
- net +5V: track 76.2 -> 23.4 mm
- net Net-(R5-Pad2): track 50.9 -> 34.9 mm
- net Net-(U2-PA3): track 48.4 -> 36.0 mm
- net GND: track 19.5 -> 28.5 mm, vias 11 -> 10
- net Net-(U1B--): track 29.4 -> 23.3 mm
- net Net-(Q1-B): track 3.15 -> 7.30 mm
- net Net-(J3-PadT): track 2.60 -> 5.89 mm
- net Net-(J5-PadT): track 0.00 -> 2.60 mm
- net Net-(J2-PadT): track 2.60 -> 0.00 mm
- net Net-(Q1-C): track 12.8 -> 10.6 mm
- net +12V: track 99.6 -> 101.3 mm
- net FAST_MIDI: track 16.2 -> 17.4 mm
- net -12V: track 56.5 -> 57.4 mm

Commit message: finished firmware for 05 melodic player
Parts:
- added R7: 18k, cynthia:R SMD 0805, F.Cu at (15.0, 32.2)
- RV1: value 10k -> 5k
- moved SW1 0.25 mm to (7.50, 62.5)
Connections:
- RV1 pad 1: Net-(U1A--) -> Net-(R7-Pad1)
Routing:
- net Net-(R7-Pad1): track 0.00 -> 13.9 mm
- net Net-(U1A--): track 22.7 -> 13.3 mm

Commit message: updated PCB
Parts:
- added D1: LED, LED_THT:LED_D5.0mm, B.Cu at (12.0, 59.2)
- added R8: 4.7k, cynthia:R SMD 0805, F.Cu at (13.0, 53.5)
- moved U2 8.75 mm to (13.2, 46.0)
- moved C3 8.75 mm to (13.0, 51.0)
- moved C8 1.95 mm to (14.5, 64.5), turned to 180 degrees
Connections:
- U2 pad 16: unconnected-(U2-PA9/PA11-Pad16) -> Net-(D1-A)
Routing:
- net Net-(D1-A): track 0.00 -> 17.4 mm, vias 0 -> 2
- net Net-(U2-PA3): track 36.0 -> 44.9 mm
- net Net-(U2-PA2): track 18.2 -> 27.0 mm
- net FAST_MIDI: track 17.4 -> 26.0 mm
- net Net-(U2-PA4): track 19.6 -> 11.9 mm
- net Net-(U2-PA7): track 15.7 -> 8.01 mm
- net Net-(U2-PA5): track 18.1 -> 10.6 mm
- net +3.3V: track 44.9 -> 51.0 mm
- net Net-(D1-K): track 0.00 -> 5.75 mm
- net SWD DATA: track 13.1 -> 7.68 mm
- net RESET: track 14.9 -> 9.90 mm
- net SWD CLOCK: track 11.3 -> 6.87 mm
- net GND: track 28.5 -> 31.9 mm, vias 10 -> 9

Commit message: 05 rev1
Parts:
- moved J4 0.50 mm to (9.00, 5.50)
- moved D1 0.50 mm to (12.5, 59.2)
- moved J5 0.50 mm to (9.00, 16.5)
- moved J3 0.25 mm to (9.00, 94.5)
Routing:
- net Net-(U2-PA2): track 27.0 -> 27.8 mm
- net Net-(U2-PA3): track 44.9 -> 44.6 mm, vias 2 -> 0

Commit message: worked on issues after building #05
Parts:
- added R10: 15k, cynthia:R SMD 0805, F.Cu at (107.5, 80.2)
- added R9: 10k, cynthia:R SMD 0805, F.Cu at (104.2, 82.0)
- R8: value 4.7k -> 2.2k
- U3: footprint Package_SO:SOIC-8_5.3x6.2mm_P1.27mm -> cynthia:SOIC-8_3.9x4.9mm_P1.27mm
- moved C1 113.3 mm to (112.0, 82.2)
- moved C2 113.3 mm to (105.0, 87.8)
- moved C3 113.3 mm to (110.0, 109.5)
- moved C4 113.3 mm to (101.0, 142.9)
- moved C5 113.3 mm to (106.0, 90.8)
- moved C6 113.3 mm to (109.5, 142.9)
- moved C7 113.3 mm to (108.5, 125.7)
- moved C8 113.3 mm to (111.5, 123.0)
- moved D1 113.3 mm to (109.5, 117.8)
- moved J1 113.3 mm to (102.0, 100.2)
- moved J2 113.3 mm to (103.5, 136.9)
- moved J3 113.3 mm to (106.0, 153.0)
- moved J4 113.3 mm to (106.0, 64.0)
- moved J5 113.3 mm to (106.0, 75.0)
- moved Q1 113.3 mm to (106.0, 152.8)
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Connections:
- R6 pad 2: Net-(U1B--) -> Net-(R10-Pad1)
- U1 pad 7: Net-(U1B--) -> Net-(R10-Pad1)
Routing:
- net Net-(R10-Pad1): track 0.00 -> 22.2 mm
- net Net-(U1B--): track 23.3 -> 11.0 mm
- net GND: track 31.9 -> 33.6 mm, vias 9 -> 10
- net Net-(U2-PA5): track 10.6 -> 9.91 mm
- net Net-(U2-PA4): track 11.9 -> 11.2 mm
Other:
- board text added: "#05: Melodic Player Rev. 2 2026 Benjamin Murauer"
